File: DIY_AWG_V1.1/temp.kicad_sch (KiCad schematic)
At the start: 21 parts, among them U9 AD9834, Y2 SG-615

Commit message: Updated AD9834_DDS, amplifier, STM32_MCU schematic
Parts:
- renumbered C42 to C61, C33 to C62, C35 to C63, C34 to C64, C36 to C65, C44 to C66, C43 to C67, C45 to C68, R24 to R37, R23 to R38, R20 to R39, TP17 to TP22, TP8 to TP23, TP9 to TP24, TP10 to TP25, TP12 to TP26, TP15 to TP27, TP16 to TP28, TP14 to TP29, U9 to U15, Y2 to Y3
