File: DIY_AWG_V1.1/untitled.kicad_sch (KiCad schematic)
At the start: 59 parts, among them U10 AMS1117-3.3, U16 TPS7A4701RGWR, U17 TPS7A4701RGWR, U18 ADP7118ARDZ-3.3-R7, U3 TPS7A3301RGWR, U6 TPS7A3301RGWR, U7 ADP7118ARDZ-3.3-R7

Commit message: Updated power_supply, AD9834_DDS schematic
Parts:
- C13, C7, C8, C87: value 2.2u -> 10u
- C79, C82, C84, C86: value 47u -> 22u
Other:
- note added: "4.7nF MLCC (2): 04023C472KAT2A (2) 2.2uF MLCC (4): CL21B335KAFNFNE (4) 10uF MLCC (4): CL10A106MO8NQNC (4) 22uF MLCC (12): GRM31CR61C226KE15L (12) 22uF Tantalum Cap (2): TAJB226K016RNJ (2) 22uF Polymer Tantalum Cap (4): T55B226M016C0070 (4) 1.5uH Inductor (2): CMLO252010F1R5MTT (2) 0.47uH Inductor (2): MNR252010TR47NT (2) 0.33uH Inductor (2): CMLO252010FR33MTT (2) 400m Resistor (6): PE0805FRF070R4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"
- note added: "Place 2 GRM31CR61C226KE15L in parallel (eff. cap - 10uF)"
- note added: "Place GRM31CR61C226KE15L & T55B226M016C0070 in parallel"
- note removed: "4.7nF MLCC (2): 04023C472KAT2A (2) 2.2uF MLCC (8): CL21B335KAFNFNE (8) 22uF MLCC (4): GRM31CR61E476ME44L (8) 47uF MLCC (4): GRM31CR61E476ME44L (4) 22uF Tantalum Cap (2): TAJB226K016RNJ (2) 22uF Polymer Tantalum Cap (4): T55B226M016C0070 (4) 1.5uH Inductor (2): CMLO252010F1R5MTT (2) 0.47uH Inductor (2): MNR252010TR47NT (2) 0.33uH Inductor (2): CMLO252010FR33MTT (2) 400m Resistor (6): PE0805FRF070R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"
- note removed: "Place 2 GRM31CR61E476ME44L in parallel"
- note removed: "Place GRM31CR61E476ME44L & T55B226M016C0070 in parallel"
Changed lines of the file:
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@@
 		)
 	)
-	(text "4.7nF MLCC (2): 04023C472KAT2A (2)\n2.2uF MLCC (8): CL21B335KAFNFNE (8)\n22uF MLCC (4): GRM31CR61E476ME44L (8)\n47uF MLCC (4): GRM31CR61E476ME44L (4)\n\n22uF Tantalum Cap (2): TAJB226K016RNJ (2)\n22uF Polymer Tantalum Cap (4): T55B226M016C0070 (4)\n\n1.5uH Inductor (2): CMLO252010F1R5MTT (2)\n0.47uH Inductor (2): MNR252010TR47NT (2)\n0.33uH Inductor (2): CMLO252010FR33MTT (2)\n\n400m Resistor (6): PE0805FRF070R4L (10)\n162k Resistor (2): PTFR0603D162KP9 (2)\n21.5k Resistor (1): ARG03DTC2152 (1)\n49.9k Resistor (1): ERA-3AED4992V (1)"
+	(text "4.7nF MLCC (2): 04023C472KAT2A (2)\n2.2uF MLCC (4): CL21B335KAFNFNE (4)\n10uF MLCC (4): CL10A106MO8NQNC (4)\n22uF MLCC (12): GRM31CR61C226KE15L (12)\n\n22uF Tantalum Cap (2): TAJB226K016RNJ (2)\n22uF Polymer Tantalum Cap (4): T55B226M016C0070 (4)\n\n1.5uH Inductor (2): CMLO252010F1R5MTT (2)\n0.47uH Inductor (2): MNR252010TR47NT (2)\n0.33uH Inductor (2): CMLO252010FR33MTT (2)\n\n400m Resistor (6): PE0805FRF070R4L (10)\n162k Resistor (2): PTFR0603D162KP9 (2)\n21.5k Resistor (1): ARG03DTC2152 (1)\n49.9k Resistor (1): ERA-3AED4992V (1)"
 		(exclude_from_sim no)
 		(at 108.966 32.258 0)
@@
 		)
 	)
-	(text "Place 2 GRM31CR61E476ME44L in parallel"
+	(text "Place 2 GRM31CR61C226KE15L in parallel\n(eff. cap - 10uF)"
 		(exclude_from_sim no)
 		(at 194.056 111.506 0)
@@
 		)
 	)
-	(text "Place GRM31CR61E476ME44L & \nT55B226M016C0070 in parallel"
+	(text "Place GRM31CR61C226KE15L & \nT55B226M016C0070 in parallel"
 		(exclude_from_sim no)
 		(at 136.652 227.838 0)
@@
 		)
 	)
-	(text "Place 2 GRM31CR61E476ME44L in parallel"
+	(text "Place 2 GRM31CR61C226KE15L in parallel\n(eff. cap - 10uF)"
 		(exclude_from_sim no)
 		(at 40.64 201.422 0)
@@
 		)
 	)
-	(text "Place GRM31CR61E476ME44L & \nT55B226M016C0070 in parallel"
+	(text "Place GRM31CR61C226KE15L & \nT55B226M016C0070 in parallel"
 		(exclude_from_sim no)
 		(at 137.922 201.93 0)
@@
 		)
 	)
-	(text "Place GRM31CR61E476ME44L & \nT55B226M016C0070 in parallel"
+	(text "Place GRM31CR61C226KE15L & \nT55B226M016C0070 in parallel"
 		(exclude_from_sim no)
 		(at 285.242 86.614 0)
@@
 		)
 	)
-	(text "Place 2 GRM31CR61E476ME44L in parallel"
+	(text "Place 2 GRM31CR61C226KE15L in parallel\n(eff. cap - 10uF)"
 		(exclude_from_sim no)
 		(at 41.656 251.714 0)
@@
 		)
 	)
-	(text "Place GRM31CR61E476ME44L & \nT55B226M016C0070 in parallel"
+	(text "Place GRM31CR61C226KE15L & \nT55B226M016C0070 in parallel"
 		(exclude_from_sim no)
 		(at 284.734 57.15 0)
@@
 		)
 	)
-	(text "Place 2 GRM31CR61E476ME44L in parallel"
+	(text "Place 2 GRM31CR61C226KE15L in parallel\n(eff. cap - 10uF)"
 		(exclude_from_sim no)
 		(at 192.786 56.388 0)
@@
 			)
 		)
-		(property "Value" "2.2u"
+		(property "Value" "10u"
 			(at 102.87 140.97 0)
 			(show_name no)
@@
 			)
 		)
-		(property "Value" "2.2u"
+		(property "Value" "10u"
 			(at 43.18 142.24 0)
 			(show_name no)
@@
 			)
 		)
-		(property "Value" "47u"
+		(property "Value" "22u"
 			(at 290.83 97.7899 0)
 			(show_name no)
@@
 			)
 		)
-		(property "Value" "47u"
+		(property "Value" "22u"
 			(at 279.4 45.7199 0)
 			(show_name no)
@@
 			)
 		)
-		(property "Value" "2.2u"
+		(property "Value" "10u"
 			(at 102.87 95.25 0)
 			(show_name no)
@@
 			)
 		)
-		(property "Value" "47u"
+		(property "Value" "22u"
 			(at 140.97 238.7599 0)
 			(show_name no)
@@
 			)
 		)
-		(property "Value" "47u"
+		(property "Value" "22u"
 			(at 128.27 190.4999 0)
 			(show_name no)
@@
 			)
 		)
-		(property "Value" "2.2u"
+		(property "Value" "10u"
 			(at 43.18 96.52 0)
 			(show_name no)

Commit message: Updated AD9834_DDS, STM32_MCU schematic
Parts:
- added TP6, TP7: TestPoint, symbol Connector:TestPoint
Connections:
- net +3V3: now also TP6.1
- net +5V: now also TP7.1
Changed lines of the file:
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@@
 	)
 	(junction
+		(at 80.01 48.26)
+		(diameter 0)
+		(color 0 0 0 0)
+	)
+	(junction
 		(at 26.67 232.41)
 		(diameter 0)
@@
 	)
 	(junction
+		(at 33.02 29.21)
+		(diameter 0)
+		(color 0 0 0 0)
+	)
+	(junction
 		(at 116.84 238.76)
 		(diameter 0)
@@
 	(wire
 		(pts
+			(xy 80.01 48.26) (xy 81.28 48.26)
+		)
+		(stroke
+			(width 0)
+			(type default)
+		)
+	)
+	(wire
+		(pts
 			(xy 182.88 38.1) (xy 185.42 38.1)
 		)
@@
 	(wire
 		(pts
+			(xy 33.02 29.21) (xy 36.83 29.21)
+		)
+		(stroke
+			(width 0)
+			(type default)
+		)
+	)
+	(wire
+		(pts
 			(xy 91.44 139.7) (xy 93.98 139.7)
 		)
@@
 	(wire
 		(pts
-			(xy 20.32 29.21) (xy 36.83 29.21)
+			(xy 20.32 29.21) (xy 33.02 29.21)
 		)
 		(stroke
@@
 	(wire
 		(pts
-			(xy 77.47 48.26) (xy 81.28 48.26)
+			(xy 77.47 48.26) (xy 80.01 48.26)
 		)
 		(stroke
@@
 	)
 	(symbol
+		(lib_id "Connector:TestPoint")
+		(at 80.01 48.26 0)
+		(unit 1)
+		(body_style 1)
+		(exclude_from_sim no)
+		(in_bom yes)
+		(on_board yes)
+		(in_pos_files yes)
+		(dnp no)
+		(property "Reference" "TP6"
+			(at 78.232 42.418 0)
+			(show_name no)
+			(do_not_autoplace no)
+			(effects
+				(font
+					(size 1.27 1.27)
+				)
+				(justify left)
+			)
+		)
+		(property "Value" "TestPoint"
+			(at 75.946 42.672 0)
+			(hide yes)
+			(show_name no)
+			(do_not_autoplace no)
+			(effects
+				(font
+					(size 1.27 1.27)
+				)
+				(justify left)
+			)
+		)
+		(property "Footprint" ""
+			(at 85.09 48.26 0)
+			(hide yes)
+			(show_name no)
+			(do_not_autoplace no)
+			(effects
+				(font
+					(size 1.27 1.27)
+				)
+			)
+		)
+		(property "Datasheet" ""
+			(at 85.09 48.26 0)
+			(hide yes)
+			(show_name no)
+			(do_not_autoplace no)
+			(effects
+				(font
+					(size 1.27 1.27)
+				)
+			)
+		)
+		(property "Description" "test point"
+			(at 80.01 48.26 0)
+			(hide yes)
+			(show_name no)
+			(do_not_autoplace no)
+			(effects
+				(font
+					(size 1.27 1.27)
+				)
+			)
+		)
+		(pin "1"
+		)
+		(instances
+			(project "DIY_AWG_V1.1"
+				(path "/508078af-d961-4af3-840e-a064a9f8d5bc/8acbd35e-0359-4140-a5a5-b9cabf9b139d"
+					(reference "TP6")
+					(unit 1)
+				)
+			)
+		)
+	)
+	(symbol
 		(lib_id "power:GND")
 		(at 212.09 105.41 0)
@@
 					(unit 1)
 				)
+			)
+		)
+	)
+	(symbol
+		(lib_id "Connector:TestPoint")
+		(at 33.02 29.21 0)
+		(unit 1)
+		(body_style 1)
+		(exclude_from_sim no)
+		(in_bom yes)
+		(on_board yes)
+		(in_pos_files yes)
+		(dnp no)
+		(property "Reference" "TP7"
+			(at 31.242 23.368 0)
+			(show_name no)
+			(do_not_autoplace no)
+			(effects
+				(font
+					(size 1.27 1.27)
+				)
+				(justify left)
+			)
+		)
+		(property "Value" "TestPoint"
+			(at 28.956 23.622 0)
+			(hide yes)
+			(show_name no)
+			(do_not_autoplace no)
+			(effects
+				(font
+					(size 1.27 1.27)
+				)
+				(justify left)
+			)
+		)
+		(property "Footprint" ""
+			(at 38.1 29.21 0)
+			(hide yes)
+			(show_name no)
+			(do_not_autoplace no)
+			(effects
+				(font
+					(size 1.27 1.27)
+				)
+			)
+		)
+		(property "Datasheet" ""
+			(at 38.1 29.21 0)
+			(hide yes)
+			(show_name no)
+			(do_not_autoplace no)
+			(effects
+				(font
+					(size 1.27 1.27)
+				)
+			)
+		)
+		(property "Description" "test point"
+			(at 33.02 29.21 0)
+			(hide yes)
+			(show_name no)
+			(do_not_autoplace no)
+			(effects
+				(font
+					(size 1.27 1.27)
+				)
+			)
+		)
+		(pin "1"
+		)
+		(instances
+			(project "DIY_AWG_V1.1"
+				(path "/508078af-d961-4af3-840e-a064a9f8d5bc/8acbd35e-0359-4140-a5a5-b9cabf9b139d"
+					(reference "TP7")
+					(unit 1)
+				)

Commit message: Updated STM32_MCU, amplifier, User_Interface, AD9834_DDS schematic
Parts:
- renumbered C33 to C1, C88 to C10, C78 to C11, C34 to C12, C87 to C14, C83 to C15, C79 to C16, C89 to C17, C84 to C18, C90 to C19, C16 to C2, C17 to C20, C80 to C21, C100 to C22, C96 to C23, C21 to C24, C81 to C25, C85 to C26, C82 to C27, C91 to C28, C86 to C29, C7 to C3, C93 to C30, C8 to C4, C92 to C5, C12 to C6, C14 to C7, C77 to C8, C19 to C9, L4 to L1, L5 to L2, L14 to L3, L12 to L4, L15 to L5, L13 to L6, R49 to R1, R48 to R10, R50 to R2, R13 to R3, R5 to R4, R9 to R5, R10 to R6, R14 to R7, R6 to R8, R15 to R9, TP7 to TP1, TP6 to TP2, TP4 to TP3, TP5 to TP4, TP30 to TP5, TP32 to TP6, TP31 to TP7, TP33 to TP8, U10 to U1, U7 to U2, U18 to U3, U3 to U4, U16 to U5, U17 to U7
Other:
- moved on the sheet: C11, C14, C15, C16, C17, C18, C19, C27, C28, C4, C7, L2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
