File: DIY_AWG_V1.1/STM32_MCU.kicad_sch (KiCad schematic)
At the start: 24 parts, among them J2 Conn_01x04_Pin, J3 Conn_01x12, SW1 SW_Push, SW2 SW_Push, U1 161N-4BVS11, U19 USBLC6-2SC6, U9 STM32G473VETx, X1 SX2M8.000B10F20TNN

Commit message: Updated AD9834_DDS, STM32_MCU schematic
Parts:
- added TP34: TestPoint, symbol Connector:TestPoint
Connections:
- net HSE_IN: now also TP34.1
Changed lines of the file:
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@@
+	)
+	(junction
+		(at 41.91 158.75)
+		(diameter 0)
+		(color 0 0 0 0)
 	)
 	(junction
@@
 	(wire
 		(pts
+			(xy 41.91 158.75) (xy 45.72 158.75)
+		)
+		(stroke
+			(width 0)
+			(type default)
+		)
+	)
+	(wire
+		(pts
 			(xy 85.09 35.56) (xy 95.25 35.56)
 		)
@@
 	(wire
 		(pts
-			(xy 38.1 158.75) (xy 45.72 158.75)
+			(xy 38.1 158.75) (xy 41.91 158.75)
 		)
 		(stroke
@@
 					(unit 1)
 				)
+			)
+		)
+	)
+	(symbol
+		(lib_id "Connector:TestPoint")
+		(at 41.91 158.75 180)
+		(unit 1)
+		(body_style 1)
+		(exclude_from_sim no)
+		(in_bom yes)
+		(on_board yes)
+		(in_pos_files yes)
+		(dnp no)
+		(property "Reference" "TP34"
+			(at 43.688 164.592 0)
+			(show_name no)
+			(do_not_autoplace no)
+			(effects
+				(font
+					(size 1.27 1.27)
+				)
+				(justify left)
+			)
+		)
+		(property "Value" "TestPoint"
+			(at 45.974 164.338 0)
+			(hide yes)
+			(show_name no)
+			(do_not_autoplace no)
+			(effects
+				(font
+					(size 1.27 1.27)
+				)
+				(justify left)
+			)
+		)
+		(property "Footprint" ""
+			(at 36.83 158.75 0)
+			(hide yes)
+			(show_name no)
+			(do_not_autoplace no)
+			(effects
+				(font
+					(size 1.27 1.27)
+				)
+			)
+		)
+		(property "Datasheet" ""
+			(at 36.83 158.75 0)
+			(hide yes)
+			(show_name no)
+			(do_not_autoplace no)
+			(effects
+				(font
+					(size 1.27 1.27)
+				)
+			)
+		)
+		(property "Description" "test point"
+			(at 41.91 158.75 0)
+			(hide yes)
+			(show_name no)
+			(do_not_autoplace no)
+			(effects
+				(font
+					(size 1.27 1.27)
+				)
+			)
+		)
+		(pin "1"
+		)
+		(instances
+			(project "DIY_AWG_V1.1"
+				(path "/508078af-d961-4af3-840e-a064a9f8d5bc/aaba8d51-2713-41de-9761-99ebb3cee83e"
+					(reference "TP34")
+					(unit 1)
+				)

Commit message: Updated STM32_MCU, amplifier, User_Interface, AD9834_DDS schematic
Parts:
- renumbered C98 to C31, C22 to C32, C23 to C33, C24 to C34, C25 to C35, C26 to C36, C27 to C37, C28 to C38, C29 to C39, C30 to C40, C31 to C41, C32 to C42, C94 to C43, J2 to J1, J3 to J2, R51 to R11, R52 to R12, R19 to R13, TP34 to TP9, U9 to U10, U19 to U8, U1 to U9

Commit message: Updated all schematics
Parts:
- removed J2: Conn_01x12, symbol Connector_Generic:Conn_01x12
- added FPC1: XW1020012-100R-002, easyeda2kicad:FPC-SMD_10P-P1.00_XW1020012-100R-001, symbol easyeda2kicad:XW1020012-100R-002
Connections:
- net +5V: now also FPC1.1, FPC1.2, FPC1.3
- net GND: now also FPC1.10, FPC1.8, FPC1.9
- net RX2: now also FPC1.5
- net RX4: now also FPC1.4
- net TX2: now also FPC1.6
- net TX4: now also FPC1.7
- no-connect marks 4 -> 6
Other:
- note removed: "Pin 11, 12 are mounting pins"
