File: DIY_AWG_V1.1/DIY_AWG_V1.1.kicad_pcb (KiCad board)
At the start: 4 copper layers, 100 x 100 mm, 253 parts, among them CN1 RH-5019, CN10 RH-5019, CN11 RH-5019, CN12 RH-5019, CN2 RH-5019, CN3 RH-5019, CN4 RH-5019, CN5 RH-5019, CN6 RH-5019, CN7 RH-5019, CN8 RH-5019, CN9 RH-5019, IC1 TLV3544IPWR, IC2 ADG704BRMZ-REEL7, IC3 LMH6505MAX, IC4 THS3091DDAR, J1 Conn_01x04_Socket, J2 Conn_01x04_Pin, J3 Conn_01x02_Pin, SW1 SW_Push, SW10 SW_Push, SW11 SW_Push, SW12 SW_Push, SW13 SW_Push, SW14 SW_Push, SW15 SW_Push, SW16 SW_Push, SW17 SW_Push, SW18 SW_Push, SW19 SW_Push, SW2 SW_Push, SW20 SW_Push, SW21 SW_Push, SW22 SW_Push, SW23 SW_Push, SW24 SW_Push, SW25 SW_Push, SW3 SW_Push, SW4 SW_Push, SW5 SW_Push, SW6 SW_Push, SW7 SW_Push, SW8 SW_Push, SW9 SW_Push, U1 AMS1117-3.3, U10 STM32G473VETx, U11 8121H-50.000NK33DRL, U12 AD9834, U13 OPA2171AIDR, U14 EC12D1564402, U15 EC12E2430404, U2 ADP7118ARDZ-3.3-R7, U3 ADP7118ARDZ-3.3-R7, U4 TPS7A3301RGWR, U5 TPS7A4701RGWR, U6 TPS7A3301RGWR, U7 TPS7A4701RGWR, U8 USBLC6-2SC6, U9 161N-4BVS11, X1 SX2M8.000B10F20TNN

Commit message: Updated PCB design
Parts:
- removed C43: 22u, Capacitor_SMD:C_1206_3216Metric
- moved C45 109.8 mm to (78.2, 50.3), turned to 0 degrees
- moved C71 108.8 mm to (164.5, 171.4)
- moved SW17 108.8 mm to (146.7, 161.0)
- moved SW18 108.8 mm to (146.7, 165.8)
- moved SW19 108.8 mm to (146.7, 170.6)
- moved SW20 108.8 mm to (146.7, 175.4)
- moved U15 108.8 mm to (170.2, 150.3)
- moved C72 108.8 mm to (164.5, 173.9)
- moved C73 108.8 mm to (164.5, 176.4)
- moved C74 108.8 mm to (164.5, 178.9)
- moved C75 108.8 mm to (164.5, 181.4)
- moved D1 108.8 mm to (168.4, 171.4)
- moved D2 108.8 mm to (168.4, 174.1)
- moved D3 108.8 mm to (168.4, 176.8)
- moved D4 108.8 mm to (168.4, 179.5)
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Other:
- board size 100 x 100 mm -> 224.5 x 101 mm

Commit message: Updated PCB schematic
Parts:
- moved CN6 111.6 mm to (53.5, 63.0), turned to 180 degrees
- moved R25 108.4 mm to (45.1, 65.6), turned to -90 degrees
- moved R23 105.4 mm to (58.9, 63.0), turned to 180 degrees
- moved R26 103.1 mm to (45.1, 69.3), turned to -90 degrees
- moved IC2 96.5 mm to (49.7, 68.5), turned to -90 degrees
- moved C48 90.7 mm to (53.7, 71.4), turned to -90 degrees
- moved R31 89.9 mm to (54.4, 68.5), turned to 0 degrees
- moved CN8 84.8 mm to (58.0, 68.5), turned to -90 degrees
- moved R20 67.8 mm to (56.7, 8.70)
- moved R21 67.8 mm to (49.7, 8.70)
- moved R22 67.8 mm to (42.7, 8.70)
- moved SW1 67.8 mm to (63.7, 0.70)
- moved SW2 67.8 mm to (56.7, 0.70)
- moved SW3 67.8 mm to (49.7, 0.70)
- moved SW4 67.8 mm to (42.7, 0.70)
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
Commit message: Updated PCB schematics
Parts:
- added C43: 22u, Capacitor_SMD:C_1206_3216Metric, F.Cu at (83.0, 47.5)
- added LED10: XL-1608SURC-06, easyeda2kicad:LED0603-RD_RED, F.Cu at (38.8, 67.5)
- added LED8: XL-1608SURC-06, easyeda2kicad:LED0603-RD_RED, F.Cu at (38.8, 61.5)
- added LED9: XL-1608SURC-06, easyeda2kicad:LED0603-RD_RED, F.Cu at (38.8, 64.5)
- added R51: 1k, Resistor_SMD:R_0603_1608Metric, F.Cu at (33.8, 61.5)
- added R52: 2k, Resistor_SMD:R_0603_1608Metric, F.Cu at (33.8, 64.5)
- added R53: 2k, Resistor_SMD:R_0603_1608Metric, F.Cu at (33.8, 67.5)
- C65, C66, C67, C68, C69, C70, R39, R40, R41, R42, R46, U13: moved to B.Cu
- moved J3 217.1 mm to (34.0, 47.2)
- moved TP24 177.4 mm to (96.0, 82.5)
- moved TP23 170.7 mm to (100.0, 89.5)
- moved R12 164.4 mm to (25.0, 83.6), turned to 0 degrees
- moved L5 163.7 mm to (25.0, 79.5), turned to 0 degrees
- moved C22 159.7 mm to (29.0, 79.3), turned to -90 degrees
- moved L2 157.7 mm to (67.5, 119.9), turned to 90 degrees
- moved C24 157.6 mm to (30.4, 84.5), turned to -90 degrees
- moved C20 155.6 mm to (32.0, 79.3), turned to 90 degrees
- moved R2 154.9 mm to (71.5, 119.6), turned to 90 degrees
- moved C2 151.8 mm to (67.7, 116.0), turned to 180 degrees
- moved U6 148.6 mm to (36.5, 82.1), turned to 180 degrees
- moved C4 146.8 mm to (67.7, 113.0), turned to 180 degrees
- moved C8 145.4 mm to (72.5, 114.3), turned to 0 degrees
- moved R13 144.9 mm to (34.1, 97.9), turned to 0 degrees
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Connections:
- FPC2 pad 5: /STM32_MCU/UART4_TX -> /STM32_MCU/UART_TX4
- FPC2 pad 6: /STM32_MCU/UART4_RX -> /STM32_MCU/UART_RX4
- J3 pad 1: /STM32_MCU/UART4_TX -> /STM32_MCU/UART_TX4
- J3 pad 2: /STM32_MCU/UART4_RX -> /STM32_MCU/UART_RX4
Other:
- board text added: "+10V"
- board text added: "+12V"
- board text added: "+3.3V"
- board text added: "+5V"
- board text added: "-10V"
- board text added: "-12V"
- board text added: "-5V"
- board text added: "GND"
