File: DIY_AWG_V1.1/DIY_AWG_V1.1.kicad_pcb (KiCad board)
At the start: 4 copper layers, 224.5 x 101 mm, 259 parts, among them CN1 RH-5019, CN10 RH-5019, CN11 RH-5019, CN12 RH-5019, CN2 RH-5019, CN3 RH-5019, CN4 RH-5019, CN5 RH-5019, CN6 RH-5019, CN7 RH-5019, CN8 RH-5019, CN9 RH-5019, IC1 TLV3544IPWR, IC2 ADG704BRMZ-REEL7, IC3 LMH6505MAX, IC4 THS3091DDAR, J1 Conn_01x04_Socket, J2 Conn_01x04_Pin, J3 Conn_01x02_Pin, SW1 SW_Push, SW10 SW_Push, SW11 SW_Push, SW12 SW_Push, SW13 SW_Push, SW14 SW_Push, SW15 SW_Push, SW16 SW_Push, SW17 SW_Push, SW18 SW_Push, SW19 SW_Push, SW2 SW_Push, SW20 SW_Push, SW21 SW_Push, SW22 SW_Push, SW23 SW_Push, SW24 SW_Push, SW25 SW_Push, SW3 SW_Push, SW4 SW_Push, SW5 SW_Push, SW6 SW_Push, SW7 SW_Push, SW8 SW_Push, SW9 SW_Push, U1 AMS1117-3.3, U10 STM32G473VETx, U11 8121H-50.000NK33DRL, U12 AD9834, U13 OPA2171AIDR, U14 EC12D1564402, U15 EC12E2430404, U2 ADP7118ARDZ-3.3-R7, U3 ADP7118ARDZ-3.3-R7, U4 TPS7A3301RGWR, U5 TPS7A4701RGWR, U6 TPS7A3301RGWR, U7 TPS7A4701RGWR, U8 USBLC6-2SC6, U9 161N-4BVS11, X1 SX2M8.000B10F20TNN

Commit message: Updated PCB schematic
Parts:
- moved CN5 1.20 mm to (41.9, 71.3)
- moved C38 0.21 mm to (86.3, 46.7)
Changed lines of the file:
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@@
 				(font
 					(size 1.27 1.27)
+					(thickness 0.15)
 				)
 			)
@@
 	(footprint "easyeda2kicad:TESTPOINT-SMD_L3.8-W2.0_RH-5019"
 		(layer "F.Cu")
-		(at 42 72.5)
+		(at 41.9 71.3)
 		(property "Reference" "CN5"
 			(at 0 -2.2 0)
@@
 	(footprint "Capacitor_SMD:C_0603_1608Metric"
 		(layer "F.Cu")
-		(at 86.5 46.65 -90)
+		(at 86.3 46.7 -90)
 		(descr "Capacitor SMD 0603 (1608 Metric), square (rectangular) end terminal, IPC-7351 nominal, (Body size source: IPC-SM-782 page 76, https://www.pcb-3d.com/wordpress/wp-content/uploads/ipc-sm-782a_amendment_1_and_2.pdf)")
 		(tags "capacitor")
@@
 				(font
 					(size 1.27 1.27)
+					(thickness 0.15)
 				)
 			)
@@
 				(font
 					(size 1.27 1.27)
+					(thickness 0.15)
 				)
 			)
@@
 	)
 	(gr_text "-5V"
-		(at 40.5 70.5 0)
+		(at 40.4 69.6 0)
 		(layer "F.SilkS")
 		(effects

Commit message: Updated PCB schematic
Parts:
- added LED11: XL-1608UBC-04, easyeda2kicad:LED0603-RD_BLUE, F.Cu at (57.2, 47.1)
- added LED12: BL-HJC36G-AV-TRB, easyeda2kicad:LED0603-R-RD_AMBER, F.Cu at (53.6, 47.1)
- added LED13: XL-1608SURC-06, easyeda2kicad:LED0603-RD_RED, F.Cu at (49.8, 47.1)
- added R54: 1k, Resistor_SMD:R_0603_1608Metric, F.Cu at (57.2, 42.1)
- added R55: 1k, Resistor_SMD:R_0603_1608Metric, F.Cu at (53.6, 42.1)
- added R56: 1k, Resistor_SMD:R_0603_1608Metric, F.Cu at (49.8, 42.1)
- C11, C24, C25, C8: moved to F.Cu
- moved TP11 8.26 mm to (47.5, 99.8), turned to -90 degrees
- moved TP12 7.39 mm to (58.7, 103.2), turned to 0 degrees
- moved LED10 6.78 mm to (39.1, 60.7)
- moved R53 6.78 mm to (34.1, 60.7)
- moved TP14 6.72 mm to (46.2, 84.9), turned to -90 degrees
- moved C31 6.69 mm to (62.0, 36.1), turned to -90 degrees
- moved CN5 6.32 mm to (41.5, 77.6), turned to 180 degrees
- moved CN3 6.30 mm to (65.3, 103.2), turned to -90 degrees
- moved TP16 5.99 mm to (41.6, 71.5), turned to -90 degrees
- moved CN2 5.88 mm to (47.5, 106.8), turned to 180 degrees
- moved C37 5.87 mm to (69.1, 36.6)
- moved CN4 5.60 mm to (46.4, 91.1), turned to 180 degrees
- moved LED8 5.11 mm to (39.1, 66.6)
- moved R51 5.11 mm to (34.1, 66.6)
- moved X1 3.32 mm to (64.7, 36.0)
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Connections:
- FPC1 pad 10: /STM32_MCU/ROW6 -> /STM32_MCU/ROW3
- FPC1 pad 11: /STM32_MCU/ROW7 -> /STM32_MCU/ROW4
- FPC1 pad 12: /STM32_MCU/COL1 -> /STM32_MCU/ROW5
- FPC1 pad 13: /STM32_MCU/COL2 -> /STM32_MCU/ROW6
- FPC1 pad 14: /STM32_MCU/COL3 -> /STM32_MCU/ROW7
- FPC1 pad 15: /STM32_MCU/ENC2_A -> /STM32_MCU/COL1
- FPC1 pad 16: /STM32_MCU/ENC2_B -> /STM32_MCU/COL2
- FPC1 pad 17: /STM32_MCU/ENC1_A -> /STM32_MCU/COL3
- FPC1 pad 18: /STM32_MCU/ENC1_B -> GND
- FPC1 pad 19: /STM32_MCU/ENC1_SW2 -> /STM32_MCU/ENC2_A
- FPC1 pad 20: /STM32_MCU/UART_RX4 -> /STM32_MCU/ENC2_B
- FPC1 pad 21: GND -> /STM32_MCU/ENC1_A
- FPC1 pad 22: GND -> /STM32_MCU/ENC1_B
- FPC1 pad 23: GND -> /STM32_MCU/ENC1_SW2
- FPC1 pad 4: /STM32_MCU/UART_TX4 -> GND
- FPC1 pad 5: /STM32_MCU/ROW1 -> /STM32_MCU/UART_TX4
- FPC1 pad 6: /STM32_MCU/ROW2 -> /STM32_MCU/UART_RX4
- FPC1 pad 7: /STM32_MCU/ROW3 -> GND
- FPC1 pad 8: /STM32_MCU/ROW4 -> /STM32_MCU/ROW1
- FPC1 pad 9: /STM32_MCU/ROW5 -> /STM32_MCU/ROW2
- SW2 pad 1: +3.3V -> +3V3
- SW3 pad 1: +3.3V -> +3V3
- SW4 pad 1: +3.3V -> +3V3
- U10 pad 32: unconnected-(U10-PB0-Pad32) -> Net-(LED12-C)
- U10 pad 33: unconnected-(U10-PB1-Pad33) -> Net-(LED13-K)
- U10 pad 55: unconnected-(U10-PD8-Pad55) -> /STM32_MCU/TX4
- U10 pad 56: /AD9834_DDS/FSELECT -> /STM32_MCU/RX4
- U10 pad 58: unconnected-(U10-PD11-Pad58) -> /AD9834_DDS/FSELECT
- U10 pad 69: /STM32_MCU/TX4 -> unconnected-(U10-PA8-Pad69)
- U10 pad 7: unconnected-(U10-PC13-Pad7) -> Net-(LED11-K)
- U10 pad 70: /STM32_MCU/RX4 -> /STM32_MCU/UART_TX4
- U10 pad 71: unconnected-(U10-PA10-Pad71) -> /STM32_MCU/UART_RX4
Routing:
- net GND: track 0.00 -> 133.4 mm, vias 0 -> 145
- net +VSW5V0: track 0.00 -> 100.8 mm, vias 0 -> 2
- net -VSW12V0: track 0.00 -> 95.3 mm, vias 0 -> 2
- net +VSW12V0: track 0.00 -> 58.7 mm, vias 0 -> 1
- net +3V3: track 0.00 -> 47.8 mm, vias 0 -> 5
- net -10.0VA: track 0.00 -> 11.4 mm, vias 0 -> 4
- net Net-(LED1-A): track 0.00 -> 11.0 mm, vias 0 -> 1
- net +10.0VA: track 0.00 -> 10.1 mm, vias 0 -> 4
- net +3.3VA_1: track 0.00 -> 9.61 mm, vias 0 -> 1
- net -5.0VA: track 0.00 -> 9.01 mm, vias 0 -> 5
- net /STM32_MCU/HSE_IN: track 0.00 -> 8.73 mm
- net Net-(U4-EN): track 0.00 -> 6.64 mm
- net Net-(U11-OUT): track 0.00 -> 6.62 mm
- net +5.0VA: track 0.00 -> 6.38 mm, vias 0 -> 4
- net Net-(U4-FB): track 0.00 -> 5.99 mm
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- added copper zone on B.Cu, net +10.0VA
- added copper zone on F.Cu, net +10.0VA
- added copper zone on B.Cu, net +3.3VA_1
- added copper zone on B.Cu, net +3V3
- added copper zone on F.Cu, net +3V3
- added copper zone on B.Cu, net +5.0VA
- added copper zone on F.Cu, net +5.0VA
- added copper zone on B.Cu, net +VSW12V0
- added copper zone on B.Cu, net +VSW5V0
- added copper zone on B.Cu, net -10.0VA
- added copper zone on F.Cu, net -10.0VA
- added copper zone on B.Cu, net -5.0VA
- added copper zone on B.Cu, net -VSW12V0
- added copper zone on B.Cu, net GND
- added copper zone on F.Cu, net GND
- added copper zone on In1.Cu, net GND
- added copper zone on In2.Cu, net GND
- added copper zone on B.Cu, net Net-(U2-EN)
- added copper zone on B.Cu, net Net-(U4-EN)
- added copper zone on B.Cu, net Net-(U5-EN)
- added copper zone on B.Cu, net Net-(U6-EN)
- added copper zone on B.Cu, net Net-(U7-EN)
Other:
- board text added: "+3V3"

Commit message: Updated PCB schematic
Parts:
- added C86: 100n, Capacitor_SMD:C_0603_1608Metric, F.Cu at (107.2, 35.1)
- added TP28: TestPoint, TestPoint:TestPoint_Pad_D1.0mm, F.Cu at (217.7, 133.6)
- added TP29: TestPoint, TestPoint:TestPoint_Pad_D1.0mm, F.Cu at (217.7, 136.7)
- C10: moved to F.Cu
- moved LED3 84.8 mm to (26.0, 58.3), turned to 0 degrees
- moved CN1 84.6 mm to (31.7, 55.8), turned to 90 degrees
- moved R7 83.1 mm to (27.6, 56.0), turned to 180 degrees
- moved C14 80.9 mm to (27.6, 54.0), turned to 180 degrees
- moved FPC1 76.5 mm to (104.4, 46.0), turned to 180 degrees
- moved TP8 75.8 mm to (40.0, 50.3), turned to -90 degrees
- moved TP7 75.6 mm to (32.7, 51.8), turned to 90 degrees
- moved U3 74.3 mm to (28.6, 49.0), turned to 180 degrees
- moved J3 74.3 mm to (108.1, 51.8), turned to 90 degrees
- moved C5 70.1 mm to (27.5, 43.1), turned to 0 degrees
- moved L3 67.7 mm to (26.7, 40.0), turned to -90 degrees
- moved C10 67.7 mm to (30.1, 43.1), turned to 180 degrees
- moved R3 65.2 mm to (29.3, 40.0), turned to -90 degrees
- moved CN7 15.3 mm to (71.9, 64.2), turned to 180 degrees
- moved C59 13.1 mm to (103.1, 73.7), turned to -90 degrees
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Connections:
- net /STM32_MCU/USB_DM renamed /STM32_MCU/USB_DN
- net Net-(U10-PB10) renamed /STM32_MCU/USER_DEF1
- net Net-(U10-PB11) renamed /STM32_MCU/USER_DEF2
- net Net-(U10-PB8) renamed /STM32_MCU/BOOT0
- FPC1 pad 10: /STM32_MCU/ROW3 -> /STM32_MCU/COL1
- FPC1 pad 11: /STM32_MCU/ROW4 -> /STM32_MCU/ROW7
- FPC1 pad 12: /STM32_MCU/ROW5 -> /STM32_MCU/ROW6
- FPC1 pad 13: /STM32_MCU/ROW6 -> /STM32_MCU/ROW5
- FPC1 pad 14: /STM32_MCU/ROW7 -> /STM32_MCU/ROW4
- FPC1 pad 15: /STM32_MCU/COL1 -> /STM32_MCU/ROW3
- FPC1 pad 16: /STM32_MCU/COL2 -> /STM32_MCU/ROW2
- FPC1 pad 17: /STM32_MCU/COL3 -> /STM32_MCU/ROW1
- FPC1 pad 19: /STM32_MCU/ENC2_A -> /STM32_MCU/ENC2_B
- FPC1 pad 20: /STM32_MCU/ENC2_B -> /STM32_MCU/ENC2_A
- FPC1 pad 5: /STM32_MCU/UART_TX4 -> /STM32_MCU/UART_RX4
- FPC1 pad 6: /STM32_MCU/UART_RX4 -> /STM32_MCU/UART_TX4
- FPC1 pad 8: /STM32_MCU/ROW1 -> /STM32_MCU/COL3
- FPC1 pad 9: /STM32_MCU/ROW2 -> /STM32_MCU/COL2
- Je1 pad 1: /AD9834_DDS/SPI2_SCLK -> /AD9834_DDS/SPI2_RESET
- Je1 pad 3: /AD9834_DDS/SPI2_CS -> /AD9834_DDS/SPI2_SCLK
- Je1 pad 4: /AD9834_DDS/SPI2_RESET -> /AD9834_DDS/SPI2_CS
- LED11 pad 1: Net-(LED11-K) -> /STM32_MCU/INIT_RUN
- LED12 pad 2: Net-(LED12-C) -> /STM32_MCU/OUT_ON
- LED13 pad 1: Net-(LED13-K) -> /STM32_MCU/ERR_ON
- U10 pad 1: /STM32_MCU/ENC2_A -> unconnected-(U10-PE2-Pad1)
- U10 pad 16: unconnected-(U10-PC1-Pad16) -> /STM32_MCU/ERR_ON
- U10 pad 17: unconnected-(U10-PC2-Pad17) -> /STM32_MCU/ENC2_B
- U10 pad 18: unconnected-(U10-PC3-Pad18) -> /STM32_MCU/OUT_ON
- U10 pad 19: unconnected-(U10-PF2-Pad19) -> /STM32_MCU/INIT_RUN
- U10 pad 2: /STM32_MCU/ENC2_B -> unconnected-(U10-PE3-Pad2)
- U10 pad 29: unconnected-(U10-PA7-Pad29) -> /AD9834_DDS/MUX1_EN
- U10 pad 30: unconnected-(U10-PC4-Pad30) -> /AD9834_DDS/MUX1_A0
- U10 pad 31: unconnected-(U10-PC5-Pad31) -> /AD9834_DDS/MUX1_A1
- U10 pad 32: Net-(LED12-C) -> unconnected-(U10-PB0-Pad32)
- U10 pad 33: Net-(LED13-K) -> unconnected-(U10-PB1-Pad33)
- U10 pad 34: unconnected-(U10-PB2-Pad34) -> /STM32_MCU/ENC2_A
- U10 pad 55: /STM32_MCU/TX4 -> unconnected-(U10-PD8-Pad55)
- U10 pad 56: /STM32_MCU/RX4 -> unconnected-(U10-PD9-Pad56)
- U10 pad 59: /AD9834_DDS/MUX1_A0 -> unconnected-(U10-PD12-Pad59)
- U10 pad 60: /AD9834_DDS/MUX1_A1 -> unconnected-(U10-PD13-Pad60)
- U10 pad 61: /AD9834_DDS/MUX1_EN -> unconnected-(U10-PD14-Pad61)
- U10 pad 7: Net-(LED11-K) -> unconnected-(U10-PC13-Pad7)
- U10 pad 79: /STM32_MCU/UART4_TX -> unconnected-(U10-PC10-Pad79)
- U10 pad 80: /STM32_MCU/UART4_RX -> unconnected-(U10-PC11-Pad80)
Routing:
- net +3V3: track 47.8 -> 230.4 mm, vias 5 -> 21
- net +3.3VA_2: track 5.65 -> 125.8 mm, vias 0 -> 14
- net /STM32_MCU/USER_DEF2: track 3.40 -> 66.0 mm, vias 0 -> 2
- net /AD9834_DDS/DAC2_OUT1: track 0.00 -> 61.6 mm, vias 0 -> 3
- net /AD9834_DDS/WAVE2_OUT: track 0.00 -> 58.3 mm, vias 0 -> 2
- net +3.3VA_1: track 9.61 -> 67.9 mm, vias 1 -> 4
- net /AD9834_DDS/SQUARE_OUT: track 0.00 -> 54.8 mm, vias 0 -> 2
- net /STM32_MCU/SWCLK: track 0.00 -> 53.8 mm, vias 0 -> 2
- net /STM32_MCU/USER_DEF1: track 2.10 -> 55.7 mm, vias 0 -> 2
- net /AD9834_DDS/MUX1_A0: track 0.00 -> 52.9 mm, vias 0 -> 2
- net /AD9834_DDS/MUX1_A1: track 0.00 -> 52.3 mm, vias 0 -> 2
- net /STM32_MCU/SWDIO: track 0.00 -> 51.8 mm, vias 0 -> 2
- net /STM32_MCU/ENC1_B: track 0.00 -> 48.7 mm, vias 0 -> 4
- net /AD9834_DDS/SPI2_CS: track 0.00 -> 47.6 mm, vias 0 -> 2
- net /AD9834_DDS/SPI2_SCLK: track 0.00 -> 47.2 mm, vias 0 -> 1
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- added copper zone on F.Cu, net +3.3VA_1
- added copper zone on B.Cu, net +3.3VA_2
- added copper zone on F.Cu, net +3.3VA_2
- added copper zone on B.Cu, net Net-(U3-EN)
- added copper zone on B.Cu, net VBUS

Commit message: Updated PCB schematic
Parts:
- moved C71 99.1 mm to (190.1, 75.6)
- moved C72 99.1 mm to (190.1, 78.1)
- moved C75 99.1 mm to (190.1, 85.6)
- moved D4 99.1 mm to (194.1, 83.8)
- moved FPC2 99.1 mm to (224.1, 41.5)
- moved SW11 99.1 mm to (161.9, 74.8)
- moved SW12 99.1 mm to (161.9, 79.7)
- moved SW19 99.1 mm to (172.4, 74.8)
- moved SW20 99.1 mm to (172.4, 79.7)
- moved TP28 99.1 mm to (243.4, 37.8)
- moved U14 99.1 mm to (195.9, 66.5)
- moved U15 99.1 mm to (195.9, 54.6)
- moved C73 99.1 mm to (190.1, 80.6)
- moved D1 99.1 mm to (194.1, 75.6)
- moved D2 99.1 mm to (194.1, 78.3)
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Routing:
- net /AD9834_DDS/MUX1_OUT: track 3.18 -> 69.8 mm
- net /AD9834_DDS/REF_SIG1: track 0.00 -> 52.0 mm, vias 0 -> 4
- net +10.0VA: track 10.1 -> 40.9 mm, vias 4 -> 13
- net /AD9834_DDS/DC_OFFSET: track 3.25 -> 32.0 mm, vias 1 -> 2
- net /Amplifier/SIG_OUT: track 0.00 -> 21.9 mm
- net +5.0VA: track 26.0 -> 47.5 mm, vias 4 -> 5
- net /Amplifier/VGA1_OUT: track 0.00 -> 19.9 mm
- net /AD9834_DDS/DC_GAIN: track 0.00 -> 14.8 mm, vias 0 -> 1
- net -5.0VA: track 33.8 -> 48.0 mm, vias 5 -> 7
- net Net-(IC4-OUT): track 0.00 -> 13.4 mm
- net (no net): track 12.7 -> 0.00 mm
- net Net-(IC4-IN-): track 0.00 -> 11.2 mm, vias 0 -> 1
- net GND: track 162.4 -> 172.1 mm, vias 196 -> 206
- net Net-(U13A-INA-): track 0.00 -> 9.23 mm
- net -10.0VA: track 11.4 -> 19.2 mm, vias 4 -> 6
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- added copper zone on F.Cu, net -5.0VA
- added copper zone on F.Cu, net /AD9834_DDS/REF_SIG1
- added copper zone on F.Cu, net Net-(CN7-Pad1)
