File: DIY_AWG_V1.1/User_Interface.kicad_sch (KiCad schematic)
At the start: 33 parts, among them SW10 SW_Push, SW11 SW_Push, SW12 SW_Push, SW13 SW_Push, SW14 SW_Push, SW15 SW_Push, SW16 SW_Push, SW17 SW_Push, SW18 SW_Push, SW19 SW_Push, SW20 SW_Push, SW21 SW_Push, SW22 SW_Push, SW23 SW_Push, SW3 SW_Push, SW4 SW_Push, SW5 SW_Push, SW6 SW_Push, SW7 SW_Push, SW8 SW_Push, SW9 SW_Push, U14 EC12D1564402, U15 EC12E2430404

Commit message: Updated schematic PCB design
Parts:
- renumbered SW8 to SW10, SW9 to SW11, SW10 to SW12, SW11 to SW13, SW12 to SW14, SW13 to SW15, SW14 to SW16, SW15 to SW17, SW16 to SW18, SW17 to SW19, SW18 to SW20, SW19 to SW21, SW20 to SW22, SW21 to SW23, SW22 to SW24, SW23 to SW25, SW3 to SW5, SW4 to SW6, SW5 to SW7, SW6 to SW8, SW7 to SW9
Changed lines of the file:
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@@
 		(in_pos_files yes)
 		(dnp no)
-		(property "Reference" "SW11"
+		(property "Reference" "SW13"
 			(at 38.1 119.38 90)
 			(show_name no)
@@
 			(project "DIY_AWG_V1.1"
 				(path "/508078af-d961-4af3-840e-a064a9f8d5bc/5e4867af-4e97-464f-8d5d-dfa2d7b207c5"
-					(reference "SW11")
+					(reference "SW13")
 					(unit 1)
 				)
@@
 		(in_pos_files yes)
 		(dnp no)
-		(property "Reference" "SW12"
+		(property "Reference" "SW14"
 			(at 38.1 132.08 90)
 			(show_name no)
@@
 			(project "DIY_AWG_V1.1"
 				(path "/508078af-d961-4af3-840e-a064a9f8d5bc/5e4867af-4e97-464f-8d5d-dfa2d7b207c5"
-					(reference "SW12")
+					(reference "SW14")
 					(unit 1)
 				)
@@
 		(in_pos_files yes)
 		(dnp no)
-		(property "Reference" "SW9"
+		(property "Reference" "SW11"
 			(at 24.13 182.88 90)
 			(show_name no)
@@
 			(project "DIY_AWG_V1.1"
 				(path "/508078af-d961-4af3-840e-a064a9f8d5bc/5e4867af-4e97-464f-8d5d-dfa2d7b207c5"
-					(reference "SW9")
+					(reference "SW11")
 					(unit 1)
 				)
@@
 		(in_pos_files yes)
 		(dnp no)
-		(property "Reference" "SW21"
+		(property "Reference" "SW23"
 			(at 52.07 157.48 90)
 			(show_name no)
@@
 			(project "DIY_AWG_V1.1"
 				(path "/508078af-d961-4af3-840e-a064a9f8d5bc/5e4867af-4e97-464f-8d5d-dfa2d7b207c5"
-					(reference "SW21")
+					(reference "SW23")
 					(unit 1)
 				)
@@
 		(in_pos_files yes)
 		(dnp no)
-		(property "Reference" "SW7"
+		(property "Reference" "SW9"
 			(at 24.13 157.48 90)
 			(show_name no)
@@
 			(project "DIY_AWG_V1.1"
 				(path "/508078af-d961-4af3-840e-a064a9f8d5bc/5e4867af-4e97-464f-8d5d-dfa2d7b207c5"
-					(reference "SW7")
+					(reference "SW9")
 					(unit 1)
 				)
@@
 		(in_pos_files yes)
 		(dnp no)
-		(property "Reference" "SW4"
+		(property "Reference" "SW6"
 			(at 24.13 119.38 90)
 			(show_name no)
@@
 			(project "DIY_AWG_V1.1"
 				(path "/508078af-d961-4af3-840e-a064a9f8d5bc/5e4867af-4e97-464f-8d5d-dfa2d7b207c5"
-					(reference "SW4")
+					(reference "SW6")
 					(unit 1)
 				)
@@
 		(in_pos_files yes)
 		(dnp no)
-		(property "Reference" "SW10"
+		(property "Reference" "SW12"
 			(at 38.1 106.68 90)
 			(show_name no)
@@
 			(project "DIY_AWG_V1.1"
 				(path "/508078af-d961-4af3-840e-a064a9f8d5bc/5e4867af-4e97-464f-8d5d-dfa2d7b207c5"
-					(reference "SW10")
+					(reference "SW12")
 					(unit 1)
 				)
@@
 		(in_pos_files yes)
 		(dnp no)
-		(property "Reference" "SW20"
+		(property "Reference" "SW22"
 			(at 52.07 144.78 90)
 			(show_name no)
@@
 			(project "DIY_AWG_V1.1"
 				(path "/508078af-d961-4af3-840e-a064a9f8d5bc/5e4867af-4e97-464f-8d5d-dfa2d7b207c5"
-					(reference "SW20")
+					(reference "SW22")
 					(unit 1)
 				)
@@
 		(in_pos_files yes)
 		(dnp no)
-		(property "Reference" "SW5"
+		(property "Reference" "SW7"
 			(at 24.13 132.08 90)
 			(show_name no)
@@
 			(project "DIY_AWG_V1.1"
 				(path "/508078af-d961-4af3-840e-a064a9f8d5bc/5e4867af-4e97-464f-8d5d-dfa2d7b207c5"
-					(reference "SW5")
+					(reference "SW7")
 					(unit 1)
 				)
@@
 		(in_pos_files yes)
 		(dnp no)
-		(property "Reference" "SW13"
+		(property "Reference" "SW15"
 			(at 38.1 144.78 90)
 			(show_name no)
@@
 			(project "DIY_AWG_V1.1"
 				(path "/508078af-d961-4af3-840e-a064a9f8d5bc/5e4867af-4e97-464f-8d5d-dfa2d7b207c5"
-					(reference "SW13")
+					(reference "SW15")
 					(unit 1)
 				)
@@
 		(in_pos_files yes)
 		(dnp no)
-		(property "Reference" "SW15"
+		(property "Reference" "SW17"
 			(at 38.1 170.18 90)
 			(show_name no)
@@
 			(project "DIY_AWG_V1.1"
 				(path "/508078af-d961-4af3-840e-a064a9f8d5bc/5e4867af-4e97-464f-8d5d-dfa2d7b207c5"
-					(reference "SW15")
+					(reference "SW17")
 					(unit 1)
 				)
@@
 		(in_pos_files yes)
 		(dnp no)
-		(property "Reference" "SW14"
+		(property "Reference" "SW16"
 			(at 38.1 157.48 90)
 			(show_name no)
@@
 			(project "DIY_AWG_V1.1"
 				(path "/508078af-d961-4af3-840e-a064a9f8d5bc/5e4867af-4e97-464f-8d5d-dfa2d7b207c5"
-					(reference "SW14")
+					(reference "SW16")
 					(unit 1)
 				)
@@
 		(in_pos_files yes)
 		(dnp no)
-		(property "Reference" "SW18"
+		(property "Reference" "SW20"
 			(at 52.07 119.38 90)
 			(show_name no)
@@
 			(project "DIY_AWG_V1.1"
 				(path "/508078af-d961-4af3-840e-a064a9f8d5bc/5e4867af-4e97-464f-8d5d-dfa2d7b207c5"
-					(reference "SW18")
+					(reference "SW20")
 					(unit 1)
 				)
@@
 		(in_pos_files yes)
 		(dnp no)
-		(property "Reference" "SW8"
+		(property "Reference" "SW10"
 			(at 24.13 170.18 90)
 			(show_name no)
@@
 			(project "DIY_AWG_V1.1"
 				(path "/508078af-d961-4af3-840e-a064a9f8d5bc/5e4867af-4e97-464f-8d5d-dfa2d7b207c5"
-					(reference "SW8")
+					(reference "SW10")
 					(unit 1)
 				)
@@
 		(in_pos_files yes)
 		(dnp no)
-		(property "Reference" "SW3"
+		(property "Reference" "SW5"
 			(at 24.13 106.68 90)
 			(show_name no)
@@
 			(project "DIY_AWG_V1.1"
 				(path "/508078af-d961-4af3-840e-a064a9f8d5bc/5e4867af-4e97-464f-8d5d-dfa2d7b207c5"
-					(reference "SW3")
+					(reference "SW5")
 					(unit 1)
 				)
@@
 		(in_pos_files yes)
 		(dnp no)
-		(property "Reference" "SW17"
+		(property "Reference" "SW19"
 			(at 52.07 106.68 90)
 			(show_name no)
@@
 			(project "DIY_AWG_V1.1"
 				(path "/508078af-d961-4af3-840e-a064a9f8d5bc/5e4867af-4e97-464f-8d5d-dfa2d7b207c5"
-					(reference "SW17")
+					(reference "SW19")
 					(unit 1)
 				)
@@
 		(in_pos_files yes)
 		(dnp no)
-		(property "Reference" "SW23"
+		(property "Reference" "SW25"
 			(at 52.07 182.88 90)
 			(show_name no)
@@
 			(project "DIY_AWG_V1.1"
 				(path "/508078af-d961-4af3-840e-a064a9f8d5bc/5e4867af-4e97-464f-8d5d-dfa2d7b207c5"
-					(reference "SW23")
+					(reference "SW25")
 					(unit 1)
 				)
@@
 		(in_pos_files yes)
 		(dnp no)
-		(property "Reference" "SW16"
+		(property "Reference" "SW18"
 			(at 38.1 182.88 90)
 			(show_name no)
@@
 			(project "DIY_AWG_V1.1"
 				(path "/508078af-d961-4af3-840e-a064a9f8d5bc/5e4867af-4e97-464f-8d5d-dfa2d7b207c5"
-					(reference "SW16")
+					(reference "SW18")
 					(unit 1)
 				)
@@
 		(in_pos_files yes)
 		(dnp no)
-		(property "Reference" "SW19"
+		(property "Reference" "SW21"
 			(at 52.07 132.08 90)
 			(show_name no)
@@
 			(project "DIY_AWG_V1.1"
 				(path "/508078af-d961-4af3-840e-a064a9f8d5bc/5e4867af-4e97-464f-8d5d-dfa2d7b207c5"
-					(reference "SW19")
+					(reference "SW21")
 					(unit 1)
 				)
@@
 		(in_pos_files yes)
 		(dnp no)
-		(property "Reference" "SW6"
+		(property "Reference" "SW8"
 			(at 24.13 144.78 90)
 			(show_name no)
@@
 			(project "DIY_AWG_V1.1"
 				(path "/508078af-d961-4af3-840e-a064a9f8d5bc/5e4867af-4e97-464f-8d5d-dfa2d7b207c5"
-					(reference "SW6")
+					(reference "SW8")
 					(unit 1)
 				)
@@
 		(in_pos_files yes)
 		(dnp no)
-		(property "Reference" "SW22"
+		(property "Reference" "SW24"
 			(at 52.07 170.18 90)
 			(show_name no)
@@
 			(project "DIY_AWG_V1.1"
 				(path "/508078af-d961-4af3-840e-a064a9f8d5bc/5e4867af-4e97-464f-8d5d-dfa2d7b207c5"
-					(reference "SW22")
+					(reference "SW24")
 					(unit 1)
 				)

Commit message: Updated PCB schematic
Other:
- note added: "UPDATE FPC CONNECTOR ARRANGEMENT"
Changed lines of the file:
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@@
+		)
+	)
+	(text "UPDATE FPC CONNECTOR ARRANGEMENT"
+		(exclude_from_sim no)
+		(at 193.802 125.73 0)
+		(effects
+			(font
+				(size 1.27 1.27)
+			)
 		)
 	)
