File: DIY_AWG_DAUGHTER_BOARD/STM32_MCU.kicad_sch (KiCad schematic)
At the start: 41 parts, among them J2 Conn_01x04_Pin, J3 Conn_01x02_Pin, SW1 SW_Push, SW2 SW_Push, SW3 SW_Push, SW4 SW_Push, U10 STM32G473VETx, U8 USBLC6-2SC6, U9 161N-4BVS11, X1 SX2M8.000B10F20TNN

Commit message: Updated project tree
Parts:
- removed FPC1: FC-10A24P11H20, easyeda2kicad:FPC-SMD_24P-P1.00_FC-10A24P11H20, symbol easyeda2kicad:FC-10A24P11H20
- removed FPC2: XW1020012-100R-002, easyeda2kicad:FPC-SMD_10P-P1.00_XW1020012-100R-001, symbol easyeda2kicad:XW1020012-100R-002
- removed J3: Conn_01x02_Pin, Connector_PinHeader_2.54mm:PinHeader_1x02_P2.54mm_Vertical, symbol Connector:Conn_01x02_Pin
- removed LED11: XL-1608UBC-04, easyeda2kicad:LED0603-RD_BLUE, symbol easyeda2kicad:XL-1608UBC-04
- removed LED12: BL-HJC36G-AV-TRB, easyeda2kicad:LED0603-R-RD_AMBER, symbol easyeda2kicad:BL-HJC36G-AV-TRB
- removed LED13: XL-1608SURC-06, easyeda2kicad:LED0603-RD_RED, symbol easyeda2kicad:XL-1608SURC-06
- removed R20, R21, R22: 5.1k, Resistor_SMD:R_0603_1608Metric, symbol Device:R
- removed R54, R55, R56: 1k, Resistor_SMD:R_0603_1608Metric, symbol Device:R
- removed SW2, SW3, SW4: SW_Push, easyeda2kicad:SW-SMD_L6.1-W3.5-LS8.6, symbol Switch:SW_Push
- removed TP28, TP29: TestPoint, TestPoint:TestPoint_Pad_D1.0mm, symbol Connector:TestPoint
Connections:
- no-connect marks 49 -> 47
Other:
- note removed: "4.7nF MLCC (2): 04023C472KAT2A (2) 100nF MLCC (9): C0603C104J3RACTU (9) 3.3uF MLCC (1): CL21B335KAFNFNE (1) 10uF MLCC (1): CL10A106KP8NNNC (1) 22uF MLCC (1): GRM31CR61C226KE15L (1) 1k Resistor (3): THD03G1001BT (3) 5.1k Resistor (3): 1RC0603F5101 (3)"
- note removed: "BOOT0"
- note removed: "Buttons and Indicators"
- note removed: "Display FPC Adapter on Daughter PCB"
- note removed: "Double Check RX4 TX4 Connection from DWIN Display"
- note removed: "ERR_ON"
- note removed: "FPC Connector on Main PCB"
- note removed: "OUT_ON"
- note removed: "RX2"
- note removed: "TX2"
- note removed: "To indicate code is running INIT_RUN"
- note removed: "User-Def 1"
- note removed: "User-Def 2"
