File: DIY_AWG_DAUGHTER_BOARD/User_Interface.kicad_sch (KiCad schematic)
At the start: 33 parts, among them SW10 SW_Push, SW11 SW_Push, SW12 SW_Push, SW13 SW_Push, SW14 SW_Push, SW15 SW_Push, SW16 SW_Push, SW17 SW_Push, SW18 SW_Push, SW19 SW_Push, SW20 SW_Push, SW21 SW_Push, SW22 SW_Push, SW23 SW_Push, SW24 SW_Push, SW25 SW_Push, SW5 SW_Push, SW6 SW_Push, SW7 SW_Push, SW8 SW_Push, SW9 SW_Push, U14 EC12D1564402, U15 EC12E2430404

Commit message: Updated project tree
Parts:
- removed C71, C72, C73, C74, C75: 100n, Capacitor_SMD:C_0603_1608Metric, symbol Device:C
- removed D1, D2, D3, D4: RL20108Q0332LC, easyeda2kicad:DFN-8_L2.0-W1.0-P0.50-BL, symbol easyeda2kicad:RL20108Q0332LC
- removed FPC3: FC-10A24P11H20, easyeda2kicad:FPC-SMD_24P-P1.00_FC-10A24P11H20, symbol easyeda2kicad:FC-10A24P11H20
- removed SW10, SW11, SW12, SW13, SW14, SW15, SW16, SW17, SW18, SW19, SW20, SW21, SW22, SW23, SW24, SW25, SW5, SW6, SW7, SW8, SW9: SW_Push, easyeda2kicad:SW-SMD_L6.1-W3.5-LS8.6, symbol Switch:SW_Push
- removed U14: EC12D1564402, easyeda2kicad:SW-TH_EC12D1564402, symbol easyeda2kicad:EC12D1564402
- removed U15: EC12E2430404, easyeda2kicad:SW-TH_ALPSALPINE_EC12EXXXX, symbol easyeda2kicad:EC12E2430404
Connections:
- no-connect marks 2 -> 0
Other:
- note removed: "100nF MLCC (5): C0603C104J3RACTU (5)"
- note removed: "6, 7 are Mounting Pads"
- note removed: "Button Matrix for User Interface"
- note removed: "D, E are Mounting Pads"
- note removed: "FPC Connector on Daughter PCB"
- note removed: "Rotary Knob for Adjusting Analog Values"
- note removed: "Rotary Knob for Navigating User Interface"
- note removed: "SW15-SW20: F1-F6 Function Buttons"
- note removed: "SW21-SW23: Extra Buttons for Wave, Mode, Utility"
- note removed: "SW3-SW14: 0-9 Numpad, Decimal Place, +-"
- note removed: "TVS Diode for Rotary Knobs and Touchscreen"
- note removed: "UPDATE FPC CONNECTOR ARRANGEMENT"
