File: DIY_AWG_DAUGHTER_BOARD/DIY_AWG_V1.1.kicad_pcb (KiCad board)
At the start: 4 copper layers, 224.5 x 101 mm, 268 parts, among them CN1 RH-5019, CN10 RH-5019, CN11 RH-5019, CN12 RH-5019, CN2 RH-5019, CN3 RH-5019, CN4 RH-5019, CN5 RH-5019, CN6 RH-5019, CN7 RH-5019, CN8 RH-5019, CN9 RH-5019, IC1 TLV3544IPWR, IC2 ADG704BRMZ-REEL7, IC3 LMH6505MAX, IC4 THS3091DDAR, J1 Conn_01x04_Socket, J2 Conn_01x04_Pin, J3 Conn_01x02_Pin, SW1 SW_Push, SW10 SW_Push, SW11 SW_Push, SW12 SW_Push, SW13 SW_Push, SW14 SW_Push, SW15 SW_Push, SW16 SW_Push, SW17 SW_Push, SW18 SW_Push, SW19 SW_Push, SW2 SW_Push, SW20 SW_Push, SW21 SW_Push, SW22 SW_Push, SW23 SW_Push, SW24 SW_Push, SW25 SW_Push, SW3 SW_Push, SW4 SW_Push, SW5 SW_Push, SW6 SW_Push, SW7 SW_Push, SW8 SW_Push, SW9 SW_Push, U1 AMS1117-3.3, U10 STM32G473VETx, U11 8121H-50.000NK33DRL, U12 AD9834, U13 OPA2171AIDR, U14 EC12D1564402, U15 EC12E2430404, U2 ADP7118ARDZ-3.3-R7, U3 ADP7118ARDZ-3.3-R7, U4 TPS7A3301RGWR, U5 TPS7A4701RGWR, U6 TPS7A3301RGWR, U7 TPS7A4701RGWR, U8 USBLC6-2SC6, U9 161N-4BVS11, X1 SX2M8.000B10F20TNN

Commit message: Updated project tree
Parts:
- removed C1, C12: 22u, easyeda2kicad:CASE-B_3528
- removed C10, C41, C42, C6: 4.7n, Capacitor_SMD:C_0402_1005Metric
- removed C11, C24, C25, C46, C8: 2.2u, Capacitor_SMD:C_0805_2012Metric
- removed C13, C14, C3, C40, C5, C53, C56, C65, C66, C69, C70: 10u, Capacitor_SMD:C_0603_1608Metric
- removed C15, C18, C2, C20, C21, C22, C23, C26, C29, C4, C43, C7, C76, C77, C80, C82, C84, C85, C9: 22u, Capacitor_SMD:C_1206_3216Metric
- removed C16, C27, C59, C61: 10n, Capacitor_SMD:C_0603_1608Metric
- removed C17, C19, C28, C30: 22u, easyeda2kicad:CAP-SMD_L3.5-W2.8-FD
- removed C31, C33, C34, C35, C36, C37, C38, C39, C45, C48, C49, C50, C52, C55, C67, C68, C78, C79, C81, C83, C86: 100n, Capacitor_SMD:C_0603_1608Metric
- removed C32: 3.3u, Capacitor_SMD:C_0805_2012Metric
- removed C44: 20p, Capacitor_SMD:C_0603_1608Metric
- removed C47: 47p, Capacitor_SMD:C_0603_1608Metric
- removed C51, C57: 510p, Capacitor_SMD:C_0603_1608Metric
- removed C54: 39p, Capacitor_SMD:C_0603_1608Metric
- removed C58: 75p, Capacitor_SMD:C_0603_1608Metric
- removed C60: 24p, Capacitor_SMD:C_0603_1608Metric
- removed C62: 82p, Capacitor_SMD:C_0603_1608Metric
- removed C63: 8.2p, Capacitor_SMD:C_0402_1005Metric
- removed C64: 68p, Capacitor_SMD:C_0603_1608Metric
- removed CN1, CN10, CN11, CN12, CN2, CN3, CN4, CN5, CN6, CN7, CN8, CN9: RH-5019, easyeda2kicad:TESTPOINT-SMD_L3.8-W2.0_RH-5019
- removed D5: TPESD1221P, easyeda2kicad:DFN1006-2L-BI
- removed IC1: TLV3544IPWR, easyeda2kicad:TSSOP-14_L5.0-W4.4-P0.65-LS6.4-BL
- removed IC2: ADG704BRMZ-REEL7, easyeda2kicad:MSOP-10_L3.0-W3.0-P0.50-LS5.0-BL
- removed IC3: LMH6505MAX, easyeda2kicad:SOP-8_L4.9-W3.9-P1.27-LS6.0-BL
- removed IC4: THS3091DDAR, easyeda2kicad:SOIC-8_L4.9-W3.9-P1.27-LS6.0-BL-EP
- removed J1: Conn_01x04_Socket, Connector_JST:JST_XH_B4B-XH-A_1x04_P2.50mm_Vertical
- removed J2, Je1: Conn_01x04_Pin, Connector_PinHeader_2.54mm:PinHeader_1x04_P2.54mm_Vertical
- removed L1, L3: 1.5u, Inductor_SMD:L_1008_2520Metric
- removed L10: 1.8u, Inductor_SMD:L_1812_4532Metric
- removed L2, L5: 0.33u, Inductor_SMD:L_1008_2520Metric
- removed L4, L6: 0.47u, Inductor_SMD:L_1008_2520Metric
- removed L7: 1u, Inductor_SMD:L_1812_4532Metric
- removed L8: 2.7u, easyeda2kicad:L_1008_2520_SLQW2520
- removed L9: 1.5u, Inductor_SMD:L_1812_4532Metric
- removed LED1, LED10, LED13, LED2, LED3, LED4, LED5, LED6, LED7, LED8, LED9: XL-1608SURC-06, easyeda2kicad:LED0603-RD_RED
- removed LED11: XL-1608UBC-04, easyeda2kicad:LED0603-RD_BLUE
- removed LED12: BL-HJC36G-AV-TRB, easyeda2kicad:LED0603-R-RD_AMBER
- removed R1, R12, R13, R2, R3, R4: 400m, Resistor_SMD:R_0805_2012Metric
- removed R10, R11, R34: 6.8k, Capacitor_SMD:C_0603_1608Metric
- removed R14, R8: 162k, Resistor_SMD:R_0603_1608Metric
- removed R15: 49.9k, Resistor_SMD:R_0603_1608Metric
- removed R16, R17, R44, R52, R53: 2k, Resistor_SMD:R_0603_1608Metric
- removed R18, R19, R20, R21, R22: 5.1k, Resistor_SMD:R_0603_1608Metric
- removed R23, R27, R31, R33, R50: 0, Resistor_SMD:R_0603_1608Metric
- removed R24, R35, R38: 200, Capacitor_SMD:C_0603_1608Metric
- removed R25, R41: 10k, Resistor_SMD:R_0603_1608Metric
- removed R26, R37, R47, R48, R5, R51, R54, R55, R56, R6, R7: 1k, Resistor_SMD:R_0603_1608Metric
- removed R28, R49: 50, Resistor_SMD:R_0603_1608Metric
- removed R29, R32: 9.53, Resistor_SMD:R_0603_1608Metric
- removed R30: 40.2, Resistor_SMD:R_0603_1608Metric
- removed R36, R39, R42: 20k, Resistor_SMD:R_0603_1608Metric
- removed R40: 30k, Resistor_SMD:R_0603_1608Metric
- removed R43: 1.3k, Resistor_SMD:R_0603_1608Metric
- removed R45: 237, Resistor_SMD:R_0603_1608Metric
- removed R46: 249, Resistor_SMD:R_0603_1608Metric
- removed R9: 21.5k, Resistor_SMD:R_0603_1608Metric
- removed RF1: KH-BNC50-3511, easyeda2kicad:ANT-TH_KH-BNC50-3511
- removed SW1, SW2, SW3, SW4: SW_Push, easyeda2kicad:SW-SMD_L6.1-W3.5-LS8.6
- removed TP1, TP10, TP11, TP12, TP13, TP14, TP15, TP16, TP17, TP18, TP19, TP2, TP20, TP21, TP22, TP23, TP24, TP25, TP26, TP27, TP3, TP4, TP5, TP6, TP7, TP8, TP9: TestPoint, TestPoint:TestPoint_Pad_D1.0mm
- removed U1: AMS1117-3.3, easyeda2kicad:SOT-223-3_L6.5-W3.4-P2.30-LS7.0-BR
- removed U10: STM32G473VETx, Package_QFP:LQFP-100_14x14mm_P0.5mm
- removed U11: 8121H-50.000NK33DRL, easyeda2kicad:OSC-SMD_4P-L2.0-W1.6-BL_SIT8008BI-72-33E-54.000000
- removed U12: AD9834, Package_SO:TSSOP-20_4.4x6.5mm_P0.65mm
- removed U13: OPA2171AIDR, easyeda2kicad:SOIC-8_L5.0-W4.0-P1.27-LS6.0-BL
- removed U2, U3: ADP7118ARDZ-3.3-R7, easyeda2kicad:SOIC-8_L4.9-W3.9-P1.27-LS6.0-BL-EP2.3
- removed U4, U6: TPS7A3301RGWR, easyeda2kicad:VQFN-20_L5.0-W5.0-P0.65-TL-EP
- removed U5, U7: TPS7A4701RGWR, easyeda2kicad:VQFN-20_L5.0-W5.0-P0.65-TL-EP
- removed U8: USBLC6-2SC6, Package_TO_SOT_SMD:SOT-23-6
- removed U9: 161N-4BVS11, easyeda2kicad:USB-C-SMD_HANELECTRICITY_161N-4XVS11
- removed X1: SX2M8.000B10F20TNN, easyeda2kicad:OSC-SMD_4P-L2.5-W2.0-BL
- moved FPC2 189.1 mm to (39.2, 2.05)
- moved TP28 187.8 mm to (58.0, 7.83)
- moved TP29 187.8 mm to (58.0, 10.9)
- moved FPC3 177.1 mm to (-1.43, 48.2)
- moved SW21 163.2 mm to (25.7, 1.91)
- moved SW23 163.2 mm to (25.7, 11.5)
- moved SW24 163.2 mm to (25.7, 16.3)
- moved SW25 163.2 mm to (25.7, 21.1)
- moved SW10 163.2 mm to (4.75, 26.0)
- moved SW11 163.2 mm to (4.75, 30.8)
- moved SW12 163.2 mm to (4.75, 35.6)
- moved SW13 163.2 mm to (15.2, 1.91)
- moved SW14 163.2 mm to (15.2, 6.71)
- moved SW15 163.2 mm to (15.2, 11.5)
- moved SW16 163.2 mm to (15.2, 16.3)
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Connections:
- net /STM32_MCU/RX4 renamed /RX4
- net /STM32_MCU/TX4 renamed /TX4
- C71 pad 1: /STM32_MCU/ENC1_A -> /ENC1_A
- C72 pad 1: /User_Interface/ENC1_SW2 -> /ENC1_SW2
- C73 pad 1: /STM32_MCU/ENC1_B -> /ENC1_B
- C74 pad 2: /STM32_MCU/ENC2_A -> /ENC2_A
- C75 pad 2: /STM32_MCU/ENC2_B -> /ENC2_B
- D1 pad 1: /STM32_MCU/ENC1_A -> /ENC1_A
- D1 pad 3: /STM32_MCU/ENC1_B -> /ENC1_B
- D1 pad 6: /STM32_MCU/ENC1_B -> /ENC1_B
- D1 pad 8: /STM32_MCU/ENC1_A -> /ENC1_A
- D2 pad 1: /User_Interface/ENC1_SW2 -> /ENC1_SW2
- D2 pad 3: /STM32_MCU/ENC2_A -> /ENC2_A
- D2 pad 6: /STM32_MCU/ENC2_A -> /ENC2_A
- D2 pad 8: /User_Interface/ENC1_SW2 -> /ENC1_SW2
- D3 pad 1: /STM32_MCU/UART_RX4 -> /UART_TX4
- D3 pad 3: /STM32_MCU/ENC2_B -> /ENC2_B
- D3 pad 6: /STM32_MCU/ENC2_B -> /ENC2_B
- D3 pad 8: /STM32_MCU/UART_RX4 -> /UART_TX4
- D4 pad 3: /STM32_MCU/UART_TX4 -> /UART_RX4
- D4 pad 6: /STM32_MCU/UART_TX4 -> /UART_RX4
- FPC1 pad 10: /STM32_MCU/COL1 -> /COL1
- FPC1 pad 11: /STM32_MCU/ROW7 -> /ROW7
- FPC1 pad 12: /STM32_MCU/ROW6 -> /ROW6
- FPC1 pad 13: /STM32_MCU/ROW5 -> /ROW5
- FPC1 pad 14: /STM32_MCU/ROW4 -> /ROW4
- FPC1 pad 15: /STM32_MCU/ROW3 -> /ROW3
- FPC1 pad 16: /STM32_MCU/ROW2 -> /ROW2
- FPC1 pad 17: /STM32_MCU/ROW1 -> /ROW1
- FPC1 pad 19: /STM32_MCU/ENC2_B -> /ENC2_B
- FPC1 pad 20: /STM32_MCU/ENC2_A -> /ENC2_A
- FPC1 pad 21: /STM32_MCU/ENC1_A -> /ENC1_A
- FPC1 pad 22: /STM32_MCU/ENC1_B -> /ENC1_B
- FPC1 pad 23: /STM32_MCU/ENC1_SW2 -> /ENC1_SW2
- FPC1 pad 5: /STM32_MCU/UART_RX4 -> /UART_RX4
- FPC1 pad 6: /STM32_MCU/UART_TX4 -> /UART_TX4
- FPC1 pad 8: /STM32_MCU/COL3 -> /COL3
- FPC1 pad 9: /STM32_MCU/COL2 -> /COL2
- FPC2 pad 5: /STM32_MCU/UART_TX4 -> /UART_TX4
- FPC2 pad 6: /STM32_MCU/UART_RX4 -> /UART_RX4
- FPC3 pad 1: +3V3 -> GND
- FPC3 pad 10: /STM32_MCU/ROW6 -> /ROW3
- FPC3 pad 11: /STM32_MCU/ROW7 -> /ROW4
- FPC3 pad 12: /STM32_MCU/COL1 -> /ROW5
- FPC3 pad 13: /STM32_MCU/COL2 -> /ROW6
- FPC3 pad 14: /STM32_MCU/COL3 -> /ROW7
- FPC3 pad 15: /STM32_MCU/ENC2_A -> /COL1
- FPC3 pad 16: /STM32_MCU/ENC2_B -> /COL2
- FPC3 pad 17: /STM32_MCU/ENC1_A -> /COL3
- FPC3 pad 18: /STM32_MCU/ENC1_B -> GND
- FPC3 pad 19: /STM32_MCU/ENC1_SW2 -> /UART_TX4
- FPC3 pad 2: +3V3 -> /ENC1_SW2
- FPC3 pad 20: /STM32_MCU/UART_TX4 -> /UART_RX4
- FPC3 pad 22: GND -> +3V3
- FPC3 pad 23: GND -> +3V3
- FPC3 pad 24: GND -> +3V3
- FPC3 pad 3: +3V3 -> /ENC1_B
- FPC3 pad 4: /STM32_MCU/UART_RX4 -> /ENC1_A
- FPC3 pad 5: /STM32_MCU/ROW1 -> /ENC2_A
- FPC3 pad 6: /STM32_MCU/ROW2 -> /ENC2_B
- FPC3 pad 7: /STM32_MCU/ROW3 -> GND
- FPC3 pad 8: /STM32_MCU/ROW4 -> /ROW1
- FPC3 pad 9: /STM32_MCU/ROW5 -> /ROW2
- J3 pad 1: /STM32_MCU/UART_TX4 -> /UART_TX4
- J3 pad 2: /STM32_MCU/UART_RX4 -> /UART_RX4
- SW10 pad 1: /STM32_MCU/COL1 -> /COL1
- SW10 pad 2: /STM32_MCU/ROW6 -> /ROW6
- SW11 pad 1: /STM32_MCU/COL1 -> /COL1
- SW11 pad 2: /STM32_MCU/ROW7 -> /ROW7
- SW12 pad 1: /STM32_MCU/COL2 -> /COL2
- SW12 pad 2: /STM32_MCU/ROW1 -> /ROW1
- SW13 pad 1: /STM32_MCU/COL2 -> /COL2
- SW13 pad 2: /STM32_MCU/ROW2 -> /ROW2
- SW14 pad 1: /STM32_MCU/COL2 -> /COL2
- SW14 pad 2: /STM32_MCU/ROW3 -> /ROW3
- SW15 pad 1: /STM32_MCU/COL2 -> /COL2
- SW15 pad 2: /STM32_MCU/ROW4 -> /ROW4
- SW16 pad 1: /STM32_MCU/COL2 -> /COL2
- SW16 pad 2: /STM32_MCU/ROW5 -> /ROW5
- SW17 pad 1: /STM32_MCU/COL2 -> /COL2
- SW17 pad 2: /STM32_MCU/ROW6 -> /ROW6
- SW18 pad 1: /STM32_MCU/COL2 -> /COL2
- SW18 pad 2: /STM32_MCU/ROW7 -> /ROW7
- SW19 pad 1: /STM32_MCU/COL3 -> /COL3
- SW19 pad 2: /STM32_MCU/ROW1 -> /ROW1
- SW20 pad 1: /STM32_MCU/COL3 -> /COL3
- SW20 pad 2: /STM32_MCU/ROW2 -> /ROW2
- SW21 pad 1: /STM32_MCU/COL3 -> /COL3
- SW21 pad 2: /STM32_MCU/ROW3 -> /ROW3
- SW22 pad 1: /STM32_MCU/COL3 -> /COL3
- SW22 pad 2: /STM32_MCU/ROW4 -> /ROW4
- SW23 pad 1: /STM32_MCU/COL3 -> /COL3
- SW23 pad 2: /STM32_MCU/ROW5 -> /ROW5
- SW24 pad 1: /STM32_MCU/COL3 -> /COL3
- SW24 pad 2: /STM32_MCU/ROW6 -> /ROW6
- SW25 pad 1: /STM32_MCU/COL3 -> /COL3
- SW25 pad 2: /STM32_MCU/ROW7 -> /ROW7
- SW5 pad 1: /STM32_MCU/COL1 -> /COL1
- SW5 pad 2: /STM32_MCU/ROW1 -> /ROW1
- SW6 pad 1: /STM32_MCU/COL1 -> /COL1
- SW6 pad 2: /STM32_MCU/ROW2 -> /ROW2
- SW7 pad 1: /STM32_MCU/COL1 -> /COL1
- SW7 pad 2: /STM32_MCU/ROW3 -> /ROW3
- SW8 pad 1: /STM32_MCU/COL1 -> /COL1
- SW8 pad 2: /STM32_MCU/ROW4 -> /ROW4
- SW9 pad 1: /STM32_MCU/COL1 -> /COL1
- SW9 pad 2: /STM32_MCU/ROW5 -> /ROW5
- U14 pad A: /STM32_MCU/ENC1_A -> /ENC1_A
- U14 pad B: /STM32_MCU/ENC1_B -> /ENC1_B
- U14 pad E: /User_Interface/ENC1_SW2 -> /ENC1_SW2
- U15 pad A: /STM32_MCU/ENC2_A -> /ENC2_A
- U15 pad B: /STM32_MCU/ENC2_B -> /ENC2_B
Routing:
- net +3V3: track 230.4 -> 0.00 mm, vias 21 -> 0
- net GND: track 172.1 -> 0.00 mm, vias 206 -> 0
- net +3.3VA_2: track 120.3 -> 0.00 mm, vias 14 -> 0
- net +VSW5V0: track 110.4 -> 0.00 mm, vias 2 -> 0
- net -VSW12V0: track 95.1 -> 0.00 mm, vias 2 -> 0
- net /AD9834_DDS/MUX1_OUT: track 69.8 -> 0.00 mm
- net +3.3VA_1: track 67.9 -> 0.00 mm, vias 4 -> 0
- net /STM32_MCU/USER_DEF2: track 66.0 -> 0.00 mm, vias 2 -> 0
- net /AD9834_DDS/DAC2_OUT1: track 61.6 -> 0.00 mm, vias 3 -> 0
- net /AD9834_DDS/WAVE2_OUT: track 58.3 -> 0.00 mm, vias 2 -> 0
- net +VSW12V0: track 57.9 -> 0.00 mm, vias 1 -> 0
- net /STM32_MCU/USER_DEF1: track 55.7 -> 0.00 mm, vias 2 -> 0
- net /AD9834_DDS/SQUARE_OUT: track 54.3 -> 0.00 mm, vias 2 -> 0
- net /STM32_MCU/SWCLK: track 53.8 -> 0.00 mm, vias 2 -> 0
- net /AD9834_DDS/MUX1_A0: track 52.8 -> 0.00 mm, vias 4 -> 0
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- removed copper zone on B.Cu, net +10.0VA
- removed copper zone on F.Cu, net +10.0VA
- removed copper zone on B.Cu, net +3.3VA_1
- removed copper zone on F.Cu, net +3.3VA_1
- removed copper zone on B.Cu, net +3.3VA_2
- removed copper zone on F.Cu, net +3.3VA_2
- removed copper zone on B.Cu, net +3V3
- removed copper zone on F.Cu, net +3V3
- removed copper zone on B.Cu, net +5.0VA
- removed copper zone on F.Cu, net +5.0VA
- removed copper zone on B.Cu, net +VSW12V0
- removed copper zone on B.Cu, net +VSW5V0
- removed copper zone on B.Cu, net -10.0VA
- removed copper zone on F.Cu, net -10.0VA
- removed copper zone on B.Cu, net -5.0VA
- removed copper zone on F.Cu, net -5.0VA
- removed copper zone on B.Cu, net -VSW12V0
- removed copper zone on F.Cu, net /AD9834_DDS/REF_SIG1
- removed copper zone on B.Cu, net GND
- removed copper zone on F.Cu, net GND
- removed copper zone on F.Cu, net Net-(CN7-Pad1)
- removed copper zone on B.Cu, net Net-(U2-EN)
- removed copper zone on B.Cu, net Net-(U3-EN)
- removed copper zone on B.Cu, net Net-(U4-EN)
- removed copper zone on B.Cu, net Net-(U5-EN)
- removed copper zone on B.Cu, net Net-(U6-EN)
- removed copper zone on B.Cu, net Net-(U7-EN)
- removed copper zone on B.Cu, net VBUS
Other:
- board size 224.5 x 101 mm -> 100 x 100 mm
- board text removed: "+10V"
- board text removed: "+12V"
- board text removed: "+3.3V"
- board text removed: "+3V3"
- board text removed: "+5V"
- board text removed: "-10V"
- board text removed: "-12V"
- board text removed: "-5V"
- board text removed: "GND"

Commit message: Edited project tree, edited daughter PCB schematic
Parts:
- removed FPC1: FC-10A24P11H20, easyeda2kicad:FPC-SMD_24P-P1.00_FC-10A24P11H20
- D1, D2, D3, D4, FPC2, FPC3: moved to B.Cu
- moved SW22 125.2 mm to (104.4, 104.1)
- moved SW21 121.3 mm to (91.1, 104.1)
- moved SW25 109.2 mm to (113.4, 86.2)
- moved H3 106.7 mm to (26.0, 118.0)
- moved FPC3 105.8 mm to (104.4, 46.0), turned to 180 degrees
- moved SW24 100.8 mm to (98.4, 86.2)
- moved SW23 94.4 mm to (83.4, 86.2)
- moved SW20 92.7 mm to (77.8, 104.1)
- moved SW16 89.7 mm to (67.8, 89.1)
- moved SW13 89.3 mm to (67.8, 74.1)
- moved SW19 88.3 mm to (64.5, 104.1)
- moved SW15 86.2 mm to (52.8, 89.1)
- moved SW18 86.0 mm to (51.1, 104.1)
- moved SW17 85.9 mm to (37.8, 104.1)
- moved SW14 85.4 mm to (37.8, 89.1)
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Connections:
- D2 pad 3: /ENC2_A -> unconnected-(D2-Pad3)
- D2 pad 6: /ENC2_A -> unconnected-(D2-Pad6)
- D3 pad 1: /UART_TX4 -> /ENC2_A
- D3 pad 8: /UART_TX4 -> /ENC2_A
- D4 pad 1: unconnected-(D4-Pad1) -> /UART_TX4
- D4 pad 8: unconnected-(D4-Pad8) -> /UART_TX4
Routing:
- net /COL1: track 0.00 -> 40.9 mm, vias 0 -> 1
- net GND: track 0.00 -> 3.31 mm, vias 0 -> 2

Commit message: Updated main PCB, daughter PCB
Parts:
- moved D3 19.9 mm to (101.7, 55.1), turned to -90 degrees
- moved J3 3.73 mm to (52.8, 51.2)
Connections:
- D1 pad 1: /ENC1_A -> /ENC1_B
- D1 pad 3: /ENC1_B -> /ENC1_A
- D1 pad 6: /ENC1_B -> /ENC1_A
- D1 pad 8: /ENC1_A -> /ENC1_B
Routing:
- net /ROW6: track 0.00 -> 231.6 mm, vias 0 -> 3
- net /ROW3: track 0.00 -> 221.3 mm, vias 0 -> 1
- net /ROW4: track 0.00 -> 192.3 mm, vias 0 -> 3
- net /ROW7: track 0.00 -> 173.7 mm, vias 0 -> 5
- net /ROW1: track 0.00 -> 151.9 mm, vias 0 -> 3
- net /ROW2: track 0.00 -> 121.4 mm, vias 0 -> 3
- net /ROW5: track 0.00 -> 118.8 mm, vias 0 -> 3
- net /COL3: track 0.00 -> 105.2 mm, vias 0 -> 8
- net /COL2: track 0.00 -> 90.9 mm, vias 0 -> 8
- net /UART_TX4: track 0.00 -> 84.2 mm, vias 0 -> 3
- net /UART_RX4: track 0.00 -> 83.4 mm, vias 0 -> 3
- net /ENC1_B: track 0.00 -> 54.1 mm, vias 0 -> 1
- net /COL1: track 40.9 -> 88.8 mm, vias 1 -> 8
- net /ENC1_A: track 0.00 -> 40.0 mm, vias 0 -> 1
- net /ENC2_A: track 0.00 -> 39.8 mm
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- added copper zone on B.Cu, net /COL1
- added copper zone on B.Cu, net /COL2
- added copper zone on B.Cu, net /COL3

Commit message: Updated daughter board and main board PCB design schematics
Parts:
- added G***: LOGO, LOGO, F.Cu at (38.8, 116.7)
- added J4: Conn_01x02_Pin, Connector_PinHeader_2.54mm:PinHeader_1x02_P2.54mm_Vertical, F.Cu at (59.6, 51.2)
- moved D2 15.5 mm to (99.0, 44.1), turned to 0 degrees
- moved D3 9.52 mm to (98.4, 64.1), turned to 0 degrees
- moved FPC3 9.02 mm to (104.4, 55.0), turned to 0 degrees
Connections:
- FPC3 pad 22: +3V3 -> +VSW5V0
- FPC3 pad 23: +3V3 -> +VSW5V0
- FPC3 pad 24: +3V3 -> +VSW5V0
Routing:
- net +VSW5V0: track 0.00 -> 82.6 mm
- net /COL3: track 105.2 -> 85.8 mm
- net /ENC2_A: track 39.8 -> 20.6 mm, vias 0 -> 2
- net /UART_RX4: track 83.4 -> 101.5 mm, vias 3 -> 1
- net /ENC2_B: track 39.2 -> 21.7 mm
- net /ROW7: track 173.7 -> 156.8 mm
- net /UART_TX4: track 84.2 -> 100.9 mm, vias 3 -> 1
- net /ROW1: track 151.9 -> 135.4 mm, vias 3 -> 1
- net /COL2: track 90.9 -> 105.3 mm, vias 8 -> 9
- net /COL1: track 88.8 -> 103.0 mm, vias 8 -> 13
- net GND: track 26.9 -> 39.1 mm, vias 18 -> 30
- net /ROW3: track 221.3 -> 232.5 mm
- net /ENC1_B: track 54.1 -> 43.4 mm, vias 1 -> 2
- net /ROW4: track 192.3 -> 183.6 mm
- net /ENC1_A: track 40.0 -> 31.5 mm, vias 1 -> 3
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- added copper zone on B.Cu, net +VSW5V0
- added copper zone on B.Cu, net /ROW6
Other:
- board text added: "AWG Daughter Board - Rev 1.1 Designed By - Stan, 2026-09-08"
- board text added: "RX"
- board text added: "RX4"
- board text added: "TX"
- board text added: "TX4"
