File: DIY_AWG_DAUGHTER_BOARD/DIY_AWG_V1.1.kicad_sch (KiCad schematic)
At the start: 4 parts

Commit message: Updated project tree
Parts:
- added C71, C72, C73, C74, C75: 100n, Capacitor_SMD:C_0603_1608Metric, symbol Device:C
- added D1, D2, D3, D4: RL20108Q0332LC, easyeda2kicad:DFN-8_L2.0-W1.0-P0.50-BL, symbol easyeda2kicad:RL20108Q0332LC
- added FPC1, FPC3: FC-10A24P11H20, easyeda2kicad:FPC-SMD_24P-P1.00_FC-10A24P11H20, symbol easyeda2kicad:FC-10A24P11H20
- added FPC2: XW1020012-100R-002, easyeda2kicad:FPC-SMD_10P-P1.00_XW1020012-100R-001, symbol easyeda2kicad:XW1020012-100R-002
- added J3: Conn_01x02_Pin, Connector_PinHeader_2.54mm:PinHeader_1x02_P2.54mm_Vertical, symbol Connector:Conn_01x02_Pin
- added SW10, SW11, SW12, SW13, SW14, SW15, SW16, SW17, SW18, SW19, SW20, SW21, SW22, SW23, SW24, SW25, SW5, SW6, SW7, SW8, SW9: SW_Push, easyeda2kicad:SW-SMD_L6.1-W3.5-LS8.6, symbol Switch:SW_Push
- added TP28, TP29: TestPoint, TestPoint:TestPoint_Pad_D1.0mm, symbol Connector:TestPoint
- added U14: EC12D1564402, easyeda2kicad:SW-TH_EC12D1564402, symbol easyeda2kicad:EC12D1564402
- added U15: EC12E2430404, easyeda2kicad:SW-TH_ALPSALPINE_EC12EXXXX, symbol easyeda2kicad:EC12E2430404
Connections:
- new net +3V3: FPC1.1, FPC1.2, FPC1.3, FPC3.22, FPC3.23, FPC3.24
- new net +VSW5V0: FPC2.1, FPC2.2, FPC2.3
- new net COL1: FPC1.10, FPC3.15, SW10.1, SW11.1, SW5.1, SW6.1, SW7.1, SW8.1, SW9.1
- new net COL2: FPC1.9, FPC3.16, SW12.1, SW13.1, SW14.1, SW15.1, SW16.1, SW17.1, SW18.1
- new net COL3: FPC1.8, FPC3.17, SW19.1, SW20.1, SW21.1, SW22.1, SW23.1, SW24.1, SW25.1
- new net ENC1_A: C71.1, D1.1, D1.8, FPC1.21, FPC3.4, U14.A
- new net ENC1_B: C73.1, D1.3, D1.6, FPC1.22, FPC3.3, U14.B
- new net ENC1_SW2: C72.1, D2.1, D2.8, FPC1.23, FPC3.2, U14.E
- new net ENC2_A: C74.2, D2.3, D2.6, FPC1.20, FPC3.5, U15.A
- new net ENC2_B: C75.2, D3.3, D3.6, FPC1.19, FPC3.6, U15.B
- new net GND: C71.2, C72.2, C73.2, C74.1, C75.1, D1.2, D1.4, D1.5, D1.7, D2.2, D2.4, D2.5, D2.7, D3.2, D3.4, D3.5, D3.7, D4.2, D4.4, D4.5, D4.7, FPC1.18, FPC1.24, FPC1.25, FPC1.26, FPC1.4, FPC1.7, FPC2.10, FPC2.8, FPC2.9, FPC3.1, FPC3.18, FPC3.21, FPC3.25, FPC3.26, FPC3.7, U14.6, U14.7, U14.C, U14.D, U15.C, U15.D, U15.E
- new net ROW1: FPC1.17, FPC3.8, SW12.2, SW19.2, SW5.2
- new net ROW2: FPC1.16, FPC3.9, SW13.2, SW20.2, SW6.2
- new net ROW3: FPC1.15, FPC3.10, SW14.2, SW21.2, SW7.2
- new net ROW4: FPC1.14, FPC3.11, SW15.2, SW22.2, SW8.2
- new net ROW5: FPC1.13, FPC3.12, SW16.2, SW23.2, SW9.2
- new net ROW6: FPC1.12, FPC3.13, SW10.2, SW17.2, SW24.2
- new net ROW7: FPC1.11, FPC3.14, SW11.2, SW18.2, SW25.2
- new net RX4: FPC2.4, TP28.1
- new net TX4: FPC2.7, TP29.1
- new net UART_RX4: D4.3, D4.6, FPC1.5, FPC2.6, FPC3.20, J3.2 (Pin_2)
- new net UART_TX4: D3.1, D3.8, FPC1.6, FPC2.5, FPC3.19, J3.1 (Pin_1)
- no-connect marks 0 -> 4
Other:
- removed sheet AD9834_DDS
- removed sheet Amplifier
- removed sheet Power_Supply
- removed sheet STM32_MCU
- removed sheet User_Interface
- note added: "100nF MLCC (5): C0603C104J3RACTU (5)"
- note added: "6, 7 are Mounting Pads"
- note added: "Button Matrix for User Interface"
- note added: "D, E are Mounting Pads"
- note added: "Display FPC Adapter on Daughter PCB"
- note added: "Double Check RX4 TX4 Connection from DWIN Display"
- note added: "FPC Connector on Daughter PCB"
- note added: "FPC Connector on Main PCB"
- note added: "RX2"
- note added: "Rotary Knob for Adjusting Analog Values"
- note added: "Rotary Knob for Navigating User Interface"
- note added: "SW15-SW20: F1-F6 Function Buttons"
- note added: "SW21-SW23: Extra Buttons for Wave, Mode, Utility"
- note added: "SW3-SW14: 0-9 Numpad, Decimal Place, +-"
- note added: "TVS Diode for Rotary Knobs and Touchscreen"
- note added: "TX2"

Commit message: Edited project tree, edited daughter PCB schematic
Parts:
- removed FPC1: FC-10A24P11H20, easyeda2kicad:FPC-SMD_24P-P1.00_FC-10A24P11H20, symbol easyeda2kicad:FC-10A24P11H20
Connections:
- net ENC2_A: now also D3.1, D3.8; no longer D2.3, D2.6
- net UART_TX4: now also D4.1, D4.8; no longer D3.1, D3.8
Other:
- note added: "SW17-SW22: F1-F6 Function Buttons"
- note added: "SW23-SW25: Extra Buttons for Wave, Mode, Utility"
- note added: "SW5-SW16: 0-9 Numpad, Decimal Place, +-"
- note removed: "FPC Connector on Main PCB"
- note removed: "SW15-SW20: F1-F6 Function Buttons"
- note removed: "SW21-SW23: Extra Buttons for Wave, Mode, Utility"
- note removed: "SW3-SW14: 0-9 Numpad, Decimal Place, +-"

Commit message: Updated main PCB, daughter PCB
Connections:
- net +3V3 is gone; now on net +VSW5V0: FPC3.22, FPC3.23, FPC3.24
- net ENC1_A: now also D1.3, D1.6; no longer D1.1, D1.8
- net ENC1_B: now also D1.1, D1.8; no longer D1.3, D1.6
Changed lines of the file:
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@@
 	)
 	(junction
+		(at 166.37 208.28)
+		(diameter 0)
+		(color 0 0 0 0)
+	)
+	(junction
+		(at 157.48 161.29)
+		(diameter 0)
+		(color 0 0 0 0)
+	)
+	(junction
 		(at 33.02 179.07)
 		(diameter 0)
@@
 	)
 	(junction
-		(at 166.37 190.5)
-		(diameter 0)
-		(color 0 0 0 0)
-	)
-	(junction
 		(at 46.99 102.87)
 		(diameter 0)
@@
 	)
 	(label "ENC1_A"
-		(at 21.59 50.8 0)
-		(effects
-			(font
-				(size 1.27 1.27)
-			)
-			(justify left bottom)
-		)
-	)
-	(label "ENC1_A"
 		(at 142.24 40.64 180)
 		(effects
@@
 		)
 	)
-	(label "ENC1_A"
-		(at 54.61 50.8 180)
-		(effects
-			(font
-				(size 1.27 1.27)
-			)
-			(justify right bottom)
-		)
-	)
 	(label "ROW6"
 		(at 154.94 135.89 0)
@@
 		)
 	)
+	(label "ENC1_B"
+		(at 21.59 50.8 0)
+		(effects
+			(font
+				(size 1.27 1.27)
+			)
+			(justify left bottom)
+		)
+	)
 	(label "ENC2_B"
 		(at 73.66 38.1 0)
@@
 		)
 	)
+	(label "ENC1_A"
+		(at 21.59 38.1 0)
+		(effects
+			(font
+				(size 1.27 1.27)
+			)
+			(justify left bottom)
+		)
+	)
 	(label "ROW7"
 		(at 154.94 138.43 0)
@@
 		)
 	)
-	(label "ENC1_B"
-		(at 21.59 38.1 0)
+	(label "ENC1_A"
+		(at 54.61 38.1 180)
 		(effects
 			(font
 				(size 1.27 1.27)
 			)
-			(justify left bottom)
+			(justify right bottom)
 		)
 	)
-	(label "COL1"
-		(at 154.94 140.97 0)
+	(label "ENC1_B"
+		(at 54.61 50.8 180)
 		(effects
 			(font
 				(size 1.27 1.27)
 			)
-			(justify left bottom)
+			(justify right bottom)
 		)
 	)
-	(label "ENC2_A"
-		(at 73.66 50.8 0)
+	(label "COL1"
+		(at 154.94 140.97 0)
 		(effects
 			(font
@@
 		)
 	)
-	(label "ENC1_B"
-		(at 54.61 38.1 180)
+	(label "ENC2_A"
+		(at 73.66 50.8 0)
 		(effects
 			(font
 				(size 1.27 1.27)
 			)
-			(justify right bottom)
+			(justify left bottom)
 		)
 	)
@@
 	)
 	(symbol
+		(lib_id "power:PWR_FLAG")
+		(at 166.37 208.28 270)
+		(unit 1)
+		(body_style 1)
+		(exclude_from_sim no)
+		(in_bom yes)
+		(on_board yes)
+		(in_pos_files yes)
+		(dnp no)
+		(fields_autoplaced yes)
+		(property "Reference" "#FLG04"
+			(at 168.275 208.28 0)
+			(hide yes)
+			(show_name no)
+			(do_not_autoplace no)
+			(effects
+				(font
+					(size 1.27 1.27)
+				)
+			)
+		)
+		(property "Value" "PWR_FLAG"
+			(at 170.18 208.2799 90)
+			(show_name no)
+			(do_not_autoplace no)
+			(effects
+				(font
+					(size 1.27 1.27)
+				)
+				(justify left)
+			)
+		)
+		(property "Footprint" ""
+			(at 166.37 208.28 0)
+			(hide yes)
+			(show_name no)
+			(do_not_autoplace no)
+			(effects
+				(font
+					(size 1.27 1.27)
+				)
+			)
+		)
+		(property "Datasheet" ""
+			(at 166.37 208.28 0)
+			(hide yes)
+			(show_name no)
+			(do_not_autoplace no)
+			(effects
+				(font
+					(size 1.27 1.27)
+				)
+			)
+		)
+		(property "Description" "Special symbol for telling ERC where power comes from"
+			(at 166.37 208.28 0)
+			(hide yes)
+			(show_name no)
+			(do_not_autoplace no)
+			(effects
+				(font
+					(size 1.27 1.27)
+				)
+			)
+		)
+		(pin "1"
+		)
+		(instances
+			(project "DIY_AWG_V1.1"
+				(path "/508078af-d961-4af3-840e-a064a9f8d5bc"
+					(reference "#FLG04")
+					(unit 1)
+				)
+			)
+		)
+	)
+	(symbol
 		(lib_id "power:GND")
 		(at 167.64 120.65 0)
@@
 	)
 	(symbol
+		(lib_id "power:+VSW")
+		(at 157.48 161.29 270)
+		(unit 1)
+		(body_style 1)
+		(exclude_from_sim no)
+		(in_bom yes)
+		(on_board yes)
+		(in_pos_files yes)
+		(dnp no)
+		(fields_autoplaced yes)
+		(property "Reference" "#PWR0117"
+			(at 153.67 161.29 0)
+			(hide yes)
+			(show_name no)
+			(do_not_autoplace no)
+			(effects
+				(font
+					(size 1.27 1.27)
+				)
+			)
+		)
+		(property "Value" "+VSW5V0"
+			(at 161.29 161.2899 90)
+			(show_name no)
+			(do_not_autoplace no)
+			(effects
+				(font
+					(size 1.27 1.27)
+				)
+				(justify left)
+			)
+		)
+		(property "Footprint" ""
+			(at 157.48 161.29 0)
+			(hide yes)
+			(show_name no)
+			(do_not_autoplace no)
+			(effects
+				(font
+					(size 1.27 1.27)
+				)
+			)
+		)
+		(property "Datasheet" ""
+			(at 157.48 161.29 0)
+			(hide yes)
+			(show_name no)
+			(do_not_autoplace no)
+			(effects
+				(font
+					(size 1.27 1.27)
+				)
+			)
+		)
+		(property "Description" "Power symbol creates a global label with name \"+VSW\""
+			(at 157.48 161.29 0)
+			(hide yes)
+			(show_name no)
+			(do_not_autoplace no)
+			(effects
+				(font
+					(size 1.27 1.27)
+				)
+			)
+		)
+		(pin "1"
+		)
+		(instances
+			(project "DIY_AWG_V1.1"
+				(path "/508078af-d961-4af3-840e-a064a9f8d5bc"
+					(reference "#PWR0117")
+					(unit 1)
+				)
+			)
+		)
+	)
+	(symbol
 		(lib_id "Switch:SW_Push")
 		(at 33.02 107.95 90)
@@
 	(symbol
 		(lib_id "power:PWR_FLAG")
-		(at 166.37 190.5 0)
+		(at 157.48 161.29 180)
 		(unit 1)
 		(body_style 1)
@@
 		(dnp no)
 		(fields_autoplaced yes)
-		(property "Reference" "#FLG02"
-			(at 166.37 188.595 0)
+		(property "Reference" "#FLG03"
+			(at 157.48 163.195 0)
 			(hide yes)
 			(show_name no)
@@
 		)
 		(property "Value" "PWR_FLAG"
-			(at 166.37 185.42 0)
+			(at 157.48 166.37 0)
 			(show_name no)
 			(do_not_autoplace no)
@@
 		)
 		(property "Footprint" ""
-			(at 166.37 190.5 0)
+			(at 157.48 161.29 0)
 			(hide yes)
 			(show_name no)
@@
 		)
 		(property "Datasheet" ""
-			(at 166.37 190.5 0)
+			(at 157.48 161.29 0)
 			(hide yes)
 			(show_name no)
@@
 		)
 		(property "Description" "Special symbol for telling ERC where power comes from"
-			(at 166.37 190.5 0)
+			(at 157.48 161.29 0)
 			(hide yes)
 			(show_name no)
@@
 			(project "DIY_AWG_V1.1"
 				(path "/508078af-d961-4af3-840e-a064a9f8d5bc"
-					(reference "#FLG02")
+					(reference "#FLG03")
 					(unit 1)
 				)
@@
 					(unit 1)
 				)
-			)
-		)
-	)
-	(symbol
-		(lib_id "power:+3V3")
-		(at 157.48 161.29 270)
-		(mirror x)
-		(unit 1)
-		(body_style 1)
-		(exclude_from_sim no)
-		(in_bom yes)
-		(on_board yes)
-		(in_pos_files yes)
-		(dnp no)
-		(fields_autoplaced yes)
-		(property "Reference" "#PWR0176"
-			(at 153.67 161.29 0)
-			(hide yes)
-			(show_name no)
-			(do_not_autoplace no)
-			(effects
-				(font
-					(size 1.27 1.27)
-				)
-			)
-		)
-		(property "Value" "+3V3"
-			(at 161.29 161.2901 90)
-			(show_name no)
-			(do_not_autoplace no)
-			(effects
-				(font
-					(size 1.27 1.27)
-				)
-				(justify left)
-			)
-		)
-		(property "Footprint" ""
-			(at 157.48 161.29 0)
-			(hide yes)
-			(show_name no)
-			(do_not_autoplace no)
-			(effects
-				(font
-					(size 1.27 1.27)
-				)
-			)
-		)
-		(property "Datasheet" ""
-			(at 157.48 161.29 0)
-			(hide yes)
-			(show_name no)
-			(do_not_autoplace no)
-			(effects
-				(font
-					(size 1.27 1.27)
-				)
-			)
-		)
-		(property "Description" "Power symbol creates a global label with name \"+3V3\""
-			(at 157.48 161.29 0)
-			(hide yes)
-			(show_name no)
-			(do_not_autoplace no)
-			(effects
-				(font
-					(size 1.27 1.27)
-				)
-			)
-		)
-		(pin "1"
-		)
-		(instances
-			(project "DIY_AWG_V1.1"
-				(path "/508078af-d961-4af3-840e-a064a9f8d5bc"
-					(reference "#PWR0176")
-					(unit 1)
-				)

Commit message: Updated daughter board and main board PCB design schematics
Parts:
- added J4: Conn_01x02_Pin, Connector_PinHeader_2.54mm:PinHeader_1x02_P2.54mm_Vertical, symbol Connector:Conn_01x02_Pin
Connections:
- net GND: now also J4.1 (Pin_1), J4.2 (Pin_2)
Changed lines of the file:
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@@
 	)
 	(junction
+		(at 198.12 208.28)
+		(diameter 0)
+		(color 0 0 0 0)
+	)
+	(junction
 		(at 58.42 76.2)
 		(diameter 0)
@@
 	(wire
 		(pts
+			(xy 198.12 208.28) (xy 198.12 209.55)
+		)
+		(stroke
+			(width 0)
+			(type default)
+		)
+	)
+	(wire
+		(pts
 			(xy 162.56 190.5) (xy 166.37 190.5)
 		)
@@
 	(wire
 		(pts
+			(xy 199.39 208.28) (xy 199.39 209.55)
+		)
+		(stroke
+			(width 0)
+			(type default)
+		)
+	)
+	(wire
+		(pts
+			(xy 195.58 207.01) (xy 198.12 207.01)
+		)
+		(stroke
+			(width 0)
+			(type default)
+		)
+	)
+	(wire
+		(pts
 			(xy 97.79 63.5) (xy 110.49 63.5)
 		)
@@
 	(wire
 		(pts
+			(xy 195.58 209.55) (xy 198.12 209.55)
+		)
+		(stroke
+			(width 0)
+			(type default)
+		)
+	)
+	(wire
+		(pts
 			(xy 22.86 140.97) (xy 33.02 140.97)
 		)
@@
 	(wire
 		(pts
+			(xy 198.12 208.28) (xy 198.12 207.01)
+		)
+		(stroke
+			(width 0)
+			(type default)
+		)
+	)
+	(wire
+		(pts
 			(xy 17.78 40.64) (xy 17.78 27.94)
 		)
@@
 	(wire
 		(pts
+			(xy 198.12 208.28) (xy 199.39 208.28)
+		)
+		(stroke
+			(width 0)
+			(type default)
+		)
+	)
+	(wire
+		(pts
 			(xy 45.72 63.5) (xy 58.42 63.5)
 		)
@@
 	)
 	(symbol
+		(lib_id "Connector:Conn_01x02_Pin")
+		(at 190.5 207.01 0)
+		(unit 1)
+		(body_style 1)
+		(exclude_from_sim no)
+		(in_bom yes)
+		(on_board yes)
+		(in_pos_files yes)
+		(dnp no)
+		(property "Reference" "J4"
+			(at 190.5 200.66 0)
+			(show_name no)
+			(do_not_autoplace no)
+			(effects
+				(font
+					(size 1.27 1.27)
+				)
+			)
+		)
+		(property "Value" "Conn_01x02_Pin"
+			(at 190.5 203.2 0)
+			(show_name no)
+			(do_not_autoplace no)
+			(effects
+				(font
+					(size 1.27 1.27)
+				)
+			)
+		)
+		(property "Footprint" "Connector_PinHeader_2.54mm:PinHeader_1x02_P2.54mm_Vertical"
+			(at 190.5 207.01 0)
+			(hide yes)
+			(show_name no)
+			(do_not_autoplace no)
+			(effects
+				(font
+					(size 1.27 1.27)
+				)
+			)
+		)
+		(property "Datasheet" ""
+			(at 190.5 207.01 0)
+			(hide yes)
+			(show_name no)
+			(do_not_autoplace no)
+			(effects
+				(font
+					(size 1.27 1.27)
+				)
+			)
+		)
+		(property "Description" "Generic connector, single row, 01x02, script generated"
+			(at 190.5 207.01 0)
+			(hide yes)
+			(show_name no)
+			(do_not_autoplace no)
+			(effects
+				(font
+					(size 1.27 1.27)
+				)
+			)
+		)
+		(pin "2"
+		)
+		(pin "1"
+		)
+		(instances
+			(project "DIY_AWG_V1.1"
+				(path "/508078af-d961-4af3-840e-a064a9f8d5bc"
+					(reference "J4")
+					(unit 1)
+				)
+			)
+		)
+	)
+	(symbol
 		(lib_id "power:GND")
 		(at 167.64 156.21 0)
@@
 					(unit 1)
 				)
+			)
+		)
+	)
+	(symbol
+		(lib_id "power:GND")
+		(at 199.39 209.55 0)
+		(unit 1)
+		(body_style 1)
+		(exclude_from_sim no)
+		(in_bom yes)
+		(on_board yes)
+		(in_pos_files yes)
+		(dnp no)
+		(property "Reference" "#PWR0118"
+			(at 199.39 215.9 0)
+			(hide yes)
+			(show_name no)
+			(do_not_autoplace no)
+			(effects
+				(font
+					(size 1.27 1.27)
+				)
+			)
+		)
+		(property "Value" "GND"
+			(at 199.39 213.614 0)
+			(hide yes)
+			(show_name no)
+			(do_not_autoplace no)
+			(effects
+				(font
+					(size 1.27 1.27)
+				)
+			)
+		)
+		(property "Footprint" ""
+			(at 199.39 209.55 0)
+			(hide yes)
+			(show_name no)
+			(do_not_autoplace no)
+			(effects
+				(font
+					(size 1.27 1.27)
+				)
+			)
+		)
+		(property "Datasheet" ""
+			(at 199.39 209.55 0)
+			(hide yes)
+			(show_name no)
+			(do_not_autoplace no)
+			(effects
+				(font
+					(size 1.27 1.27)
+				)
+			)
+		)
+		(property "Description" "Power symbol creates a global label with name \"GND\" , ground"
+			(at 199.39 209.55 0)
+			(hide yes)
+			(show_name no)
+			(do_not_autoplace no)
+			(effects
+				(font
+					(size 1.27 1.27)
+				)
+			)
+		)
+		(pin "1"
+		)
+		(instances
+			(project "DIY_AWG_V1.1"
+				(path "/508078af-d961-4af3-840e-a064a9f8d5bc"
+					(reference "#PWR0118")
+					(unit 1)
+				)
