File: DIY_AWG_MAIN_BOARD/amplfier.kicad_sch (KiCad schematic)
At the start: 23 parts, among them CN10 RH-5019, IC3 LMH6505MAX, IC4 THS3091DDAR

Commit message: Updated main board schematic and design
Parts:
- added C71, C72, C73: 100n, Capacitor_SMD:C_0603_1608Metric, symbol Device:C
Connections:
- net DC_GAIN: now also C73.1
- net DC_OFFSET: now also C71.1
- net GND: now also C71.2, C72.1, C73.2
- net REF_SIG1: now also C72.2
Other:
- note added: "100nF MLCC (7): C0603C104J3RACTU (7) 6.8uF MLCC (6): GRM31CR61C226KE15L (6) 0 Resistor (1): RK73Z1JRTTD (1) 50 Resistor (1): RT0603BRD0750RL (1) 237 Resistor (1): ARG03BTC2370 (1) 249 Resistor (1): AR03BTCX2490 (1) 1k Resistor (1): THD03G1001BT (1) 1.3k Resistor (1): RT0603BRE071K3L (1) 2k Resistor (1): AR03BTDX2001 (1)"
- note removed: "100nF MLCC (4): C0603C104J3RACTU (4) 6.8uF MLCC (6): GRM31CR61C226KE15L (6) 0 Resistor (1): RK73Z1JRTTD (1) 50 Resistor (1): RT0603BRD0750RL (1) 237 Resistor (1): ARG03BTC2370 (1) 249 Resistor (1): AR03BTCX2490 (1) 1k Resistor (1): THD03G1001BT (1) 1.3k Resistor (1): RT0603BRE071K3L (1) 2k Resistor (1): AR03BTDX2001 (1)"
- moved on the sheet: C76, C77, C78, C79, C80, C81, C82, C83, C84, C85, CN10, D5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
