File: DIY_AWG_MAIN_BOARD/AD9834_DDS.kicad_sch (KiCad schematic)
At the start: 72 parts, among them CN11 RH-5019, CN12 RH-5019, CN6 RH-5019, CN7 RH-5019, CN8 RH-5019, CN9 RH-5019, IC1 TLV3544IPWR, IC2 ADG704BRMZ-REEL7, U11 8121H-50.000NK33DRL, U12 AD9834, U13 OPA2171AIDR

Commit message: Updated main board schematic and PCB
Parts:
- C46: value 2.2u -> 3.3u
- L7: Component Name 1812CS-102XJLC -> 1812CS-102XGLC
Changed lines of the file:
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@@
 			)
 		)
-		(property "Value" "2.2u"
+		(property "Value" "3.3u"
 			(at 70.104 77.47 0)
 			(show_name no)
@@
 			)
 		)
-		(property "Component Name" "1812CS-102XJLC"
+		(property "Component Name" "1812CS-102XGLC"
 			(at 90.424 40.132 90)
 			(show_name no)
