File: DIY_AWG_MAIN_BOARD/DIY_AWG_V1.1.kicad_pcb (KiCad board)
At the start: 4 copper layers, 100 x 100 mm, 235 parts, among them CN1 RH-5019, CN10 RH-5019, CN11 RH-5019, CN12 RH-5019, CN2 RH-5019, CN3 RH-5019, CN4 RH-5019, CN5 RH-5019, CN6 RH-5019, CN7 RH-5019, CN8 RH-5019, CN9 RH-5019, IC1 TLV3544IPWR, IC2 ADG704BRMZ-REEL7, IC3 LMH6505MAX, IC4 THS3091DDAR, J1 Conn_01x04_Socket, J2 Conn_01x04_Pin, SW1 SW_Push, SW2 SW_Push, SW3 SW_Push, SW4 SW_Push, U1 AMS1117-3.3, U10 STM32G473VETx, U11 8121H-50.000NK33DRL, U12 AD9834, U13 OPA2171AIDR, U2 ADP7118ARDZ-3.3-R7, U3 ADP7118ARDZ-3.3-R7, U4 TPS7A3301RGWR, U5 TPS7A4701RGWR, U6 TPS7A3301RGWR, U7 TPS7A4701RGWR, U8 USBLC6-2SC6, U9 161N-4BVS11, X1 SX2M8.000B10F20TNN

Commit message: Updated main board schematic and PCB
Connections:
- IC4 pad : GND -> (no net)
Changed lines of the file:
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@@
 			(layers "*.Cu" "*.Paste" "*.Mask")
 			(remove_unused_layers no)
-			(net "GND")
 		)
 		(pad "" thru_hole circle
@@
 			(layers "*.Cu" "*.Mask")
 			(remove_unused_layers no)
-			(net "GND")
 		)
 		(pad "" thru_hole circle
@@
 			(layers "*.Cu" "*.Paste" "*.Mask")
 			(remove_unused_layers no)
-			(net "GND")
 		)
 		(pad "" thru_hole circle
@@
 			(layers "*.Cu" "*.Paste" "*.Mask")
 			(remove_unused_layers no)
-			(net "GND")
 		)
 		(pad "1" smd oval
@@
 	)
 	(segment
-		(start 37.315 63.7)
-		(end 37.325 63.71)
-		(width 0.3)
-		(layer "F.Cu")
-		(net "Net-(LED9-K)")
-	)
-	(segment
-		(start 34.925 63.7)
-		(end 37.315 63.7)
-		(width 0.3)
-		(layer "F.Cu")
-		(net "Net-(LED9-K)")
-	)
-	(segment
-		(start 100.2 32.395)
-		(end 100.2 29.6)
-		(width 0.3)
-		(layer "F.Cu")
-		(net "Net-(U9-CC2)")
-	)
-	(segment
-		(start 99.795 32.8)
-		(end 100.2 32.395)
-		(width 0.3)
-		(layer "F.Cu")
-		(net "Net-(U9-CC2)")
-	)
-	(segment
 		(start 87.86 78.315)
 		(end 87.89 78.285)
@@
 	)
 	(segment
+		(start 37.315 63.7)
+		(end 37.325 63.71)
+		(width 0.3)
+		(layer "F.Cu")
+		(net "Net-(LED9-K)")
+	)
+	(segment
+		(start 34.925 63.7)
+		(end 37.315 63.7)
+		(width 0.3)
+		(layer "F.Cu")
+		(net "Net-(LED9-K)")
+	)
+	(segment
+		(start 100.2 32.395)
+		(end 100.2 29.6)
+		(width 0.3)
+		(layer "F.Cu")
+		(net "Net-(U9-CC2)")
+	)
+	(segment
+		(start 99.795 32.8)
+		(end 100.2 32.395)
+		(width 0.3)
+		(layer "F.Cu")
+		(net "Net-(U9-CC2)")
+	)
+	(segment
