File: DIY_AWG_MAIN_BOARD/untitled.kicad_sch (KiCad schematic)
At the start: 95 parts, among them CN1 RH-5019, CN2 RH-5019, CN3 RH-5019, CN4 RH-5019, CN5 RH-5019, J1 Conn_01x04_Socket, U1 AMS1117-3.3, U2 ADP7118ARDZ-3.3-R7, U3 ADP7118ARDZ-3.3-R7, U4 TPS7A3301RGWR, U5 TPS7A4701RGWR, U6 TPS7A3301RGWR, U7 TPS7A4701RGWR

Commit message: Updated main board schematic and design
Parts:
- removed C17, C19, C28, C30: 22u, easyeda2kicad:CAP-SMD_L3.5-W2.8-FD, symbol Device:C_Polarized
- added C17, C19, C28, C30: 100u, Capacitor_SMD:C_1210_3225Metric, symbol Device:C
Connections:
- net +10.0VA: now also C17.1
- net +5.0VA: now also C28.1
- net -10.0VA: now also C19.1
- net -5.0VA: now also C30.1
- net GND: now also C17.2, C19.2, C28.2, C30.2
Other:
- note added: "4.7nF MLCC (2): 04023C472KAT2A (2) 2.2uF MLCC (4): CL21B335KAFNFNE (4) 10uF MLCC (4): CL10A106MO8NQNC (4) 22uF MLCC (12): GRM31CR61C226KE15L (12) 100uF MLCC (4): EMK325ABJ107MM-T (4) 22uF Tantalum Cap (2): TAJB226K016RNJ (2) 1.5uH Inductor (2): CMLO252010F1R5MTT (2) 0.47uH Inductor (2): MNR252010TR47NT (2) 0.33uH Inductor (2): CMLO252010FR33MTT (2) 400m Resistor (6): PE0805FRF070R4L (6) 1k Resist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"
- note added: "Place GRM31CR61C226KE15L & EMK325ABJ107MM-T in parallel"
- note removed: "4.7nF MLCC (2): 04023C472KAT2A (2) 2.2uF MLCC (4): CL21B335KAFNFNE (4) 10uF MLCC (4): CL10A106MO8NQNC (4) 22uF MLCC (12): GRM31CR61C226KE15L (12) 22uF Tantalum Cap (2): TAJB226K016RNJ (2) 22uF Polymer Tantalum Cap (4): T55B226M016C0070 (4) 1.5uH Inductor (2): CMLO252010F1R5MTT (2) 0.47uH Inductor (2): MNR252010TR47NT (2) 0.33uH Inductor (2): CMLO252010FR33MTT (2) 400m Resistor (6): PE0805FRF070R4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"
- note removed: "Place GRM31CR61C226KE15L & T55B226M016C0070 in parallel"

Commit message: Updated main board schematic and PCB
Parts:
- C11, C24, C25, C8: value 2.2u -> 3.3u
Other:
- note added: "4.7nF MLCC (2): 04023C472KAT2A (2) 3.3uF MLCC (4): CL21B335KAFNFNE (4) 10uF MLCC (4): CL10A106MO8NQNC (4) 22uF MLCC (12): GRM31CR61C226KE15L (12) 100uF MLCC (4): EMK325ABJ107MM-T (4) 22uF Tantalum Cap (2): TAJB226K016RNJ (2) 1.5uH Inductor (2): CMLO252010F1R5MTT (2) 0.47uH Inductor (2): MNR252010TR47NT (2) 0.33uH Inductor (2): CMLO252010FR33MTT (2) 400m Resistor (6): PE0805FRF070R4L (6) 1k Resist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"
- note removed: "4.7nF MLCC (2): 04023C472KAT2A (2) 2.2uF MLCC (4): CL21B335KAFNFNE (4) 10uF MLCC (4): CL10A106MO8NQNC (4) 22uF MLCC (12): GRM31CR61C226KE15L (12) 100uF MLCC (4): EMK325ABJ107MM-T (4) 22uF Tantalum Cap (2): TAJB226K016RNJ (2) 1.5uH Inductor (2): CMLO252010F1R5MTT (2) 0.47uH Inductor (2): MNR252010TR47NT (2) 0.33uH Inductor (2): CMLO252010FR33MTT (2) 400m Resistor (6): PE0805FRF070R4L (6) 1k Resist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"
Changed lines of the file:
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@@
 		)
 	)
-	(text "4.7nF MLCC (2): 04023C472KAT2A (2)\n2.2uF MLCC (4): CL21B335KAFNFNE (4)\n10uF MLCC (4): CL10A106MO8NQNC (4)\n22uF MLCC (12): GRM31CR61C226KE15L (12)\n100uF MLCC (4): EMK325ABJ107MM-T (4)\n\n22uF Tantalum Cap (2): TAJB226K016RNJ (2)\n\n1.5uH Inductor (2): CMLO252010F1R5MTT (2)\n0.47uH Inductor (2): MNR252010TR47NT (2)\n0.33uH Inductor (2): CMLO252010FR33MTT (2)\n\n400m Resistor (6): PE0805FRF070R4L (6)\n1k Resistor (4): THD03G1001BT (4)\n2k Resistor (2): AR03BTDX2001 (2)\n162k Resistor (2): PTFR0603D162KP9 (2)\n21.5k Resistor (1): ARG03DTC2152 (1)\n49.9k Resistor (1): ERA-3AED4992V (1)"
+	(text "4.7nF MLCC (2): 04023C472KAT2A (2)\n3.3uF MLCC (4): CL21B335KAFNFNE (4)\n10uF MLCC (4): CL10A106MO8NQNC (4)\n22uF MLCC (12): GRM31CR61C226KE15L (12)\n100uF MLCC (4): EMK325ABJ107MM-T (4)\n\n22uF Tantalum Cap (2): TAJB226K016RNJ (2)\n\n1.5uH Inductor (2): CMLO252010F1R5MTT (2)\n0.47uH Inductor (2): MNR252010TR47NT (2)\n0.33uH Inductor (2): CMLO252010FR33MTT (2)\n\n400m Resistor (6): PE0805FRF070R4L (6)\n1k Resistor (4): THD03G1001BT (4)\n2k Resistor (2): AR03BTDX2001 (2)\n162k Resistor (2): PTFR0603D162KP9 (2)\n21.5k Resistor (1): ARG03DTC2152 (1)\n49.9k Resistor (1): ERA-3AED4992V (1)"
 		(exclude_from_sim no)
 		(at 118.11 71.12 0)
@@
 			)
 		)
-		(property "Value" "2.2u"
+		(property "Value" "3.3u"
 			(at 68.834 218.44 0)
 			(show_name no)
@@
 			)
 		)
-		(property "Value" "2.2u"
+		(property "Value" "3.3u"
 			(at 228.854 48.26 0)
 			(show_name no)
@@
 			)
 		)
-		(property "Value" "2.2u"
+		(property "Value" "3.3u"
 			(at 57.404 267.97 0)
 			(show_name no)
@@
 			)
 		)
-		(property "Value" "2.2u"
+		(property "Value" "3.3u"
 			(at 222.504 101.6 0)
 			(show_name no)
